File: TMCM_1260_alternative/TMCM_1260_alternative.kicad_pcb (KiCad board)
At the start: 2 copper layers, 60 x 60 mm, 29 parts, among them J1 Motor, J2 CAN, J3 I/O, J4 Power, J7 Conn_01x05, U1 LMZM23600V3SILR, U2 STM32F091CCTx, U3 TCAN337, U4 TMC5160A-TA-T, Y1 Crystal_Small

Commit message: not finished
Parts:
- added C12: 470nF, Capacitor_SMD:C_0805_2012Metric, F.Cu at (139.7, 120.2)
- added C13: 470nF, Capacitor_SMD:C_0805_2012Metric, F.Cu at (139.7, 123.2)
- added C14: 470nF, Capacitor_SMD:C_0805_2012Metric, F.Cu at (139.7, 126.2)
- added C15: 470nF, Capacitor_SMD:C_0805_2012Metric, F.Cu at (139.7, 129.2)
- added C16: 2n2, Capacitor_SMD:C_0603_1608Metric, F.Cu at (106.9, 112.4)
- added C17: 1n, 100V, Capacitor_SMD:C_0603_1608Metric, F.Cu at (51.9, 87.7)
- added C18: 1n, 100V, Capacitor_SMD:C_0603_1608Metric, F.Cu at (51.9, 90.2)
- added C19: 1n, 100V, Capacitor_SMD:C_0603_1608Metric, F.Cu at (51.9, 92.7)
- added C20: 1n, 100V, Capacitor_SMD:C_0603_1608Metric, F.Cu at (51.9, 95.2)
- added C21: 4u7, Capacitor_SMD:C_0805_2012Metric, F.Cu at (61.4, 103.0)
- added C22: 330u, Capacitor_THT:CP_Radial_D10.0mm_P5.00mm, F.Cu at (39.9, 78.3)
- added C23: 330u, Capacitor_THT:CP_Radial_D10.0mm_P5.00mm, F.Cu at (39.9, 89.8)
- added C24: 330u, Capacitor_THT:CP_Radial_D10.0mm_P5.00mm, F.Cu at (39.9, 101.4)
- added C25: 2n2, Capacitor_SMD:C_0603_1608Metric, F.Cu at (103.8, 112.4)
- added C26: 100n, Capacitor_SMD:C_0603_1608Metric, F.Cu at (51.9, 100.3)
- added C27: 10u, Capacitor_SMD:C_0805_2012Metric, F.Cu at (61.4, 106.0)
- added C28: 10u, Capacitor_SMD:C_0805_2012Metric, F.Cu at (61.4, 109.0)
- added C29: 470n, Capacitor_SMD:C_0603_1608Metric, F.Cu at (55.9, 85.2)
- added C30: 470n, Capacitor_SMD:C_0603_1608Metric, F.Cu at (55.9, 87.7)
- added C31: 100n, 16V, Capacitor_SMD:C_0603_1608Metric, F.Cu at (55.9, 90.2)
- added C32: 22n, 100V, Capacitor_SMD:C_0603_1608Metric, F.Cu at (55.9, 92.7)
- added C33: 470n, Capacitor_SMD:C_0603_1608Metric, F.Cu at (55.9, 95.2)
- added C34: 1n, 100V, Capacitor_SMD:C_0603_1608Metric, F.Cu at (55.9, 97.8)
- added C35: 1n, 100V, Capacitor_SMD:C_0603_1608Metric, F.Cu at (55.9, 100.3)
- added C36: 100n, Capacitor_SMD:C_0603_1608Metric, F.Cu at (59.9, 85.2)
- added D4: schotty diode, Diode_SMD:D_MicroSMP_AK, F.Cu at (57.0, 102.9)
- added D5: schotty diode, Diode_SMD:D_MicroSMP_AK, F.Cu at (57.0, 105.8)
- added D6: schotty diode, Diode_SMD:D_MicroSMP_AK, F.Cu at (57.0, 108.6)
- added D7: schotty diode, Diode_SMD:D_MicroSMP_AK, F.Cu at (57.0, 111.5)
- added Q1: NVMFD5C650NLT1G, NTMFD5C446NLT1G:NVMFD5C446NLWFT1G, F.Cu at (81.8, 114.4)
- added Q2: NVMFD5C650NLT1G, NTMFD5C446NLT1G:NVMFD5C446NLWFT1G, F.Cu at (81.7, 104.4)
- added Q3: NVMFD5C650NLT1G, NTMFD5C446NLT1G:NVMFD5C446NLWFT1G, F.Cu at (81.7, 94.5)
- added Q4: NVMFD5C650NLT1G, NTMFD5C446NLT1G:NVMFD5C446NLWFT1G, F.Cu at (81.7, 84.4)
- added R10: 15, Resistor_SMD:R_1206_3216Metric, F.Cu at (88.9, 105.7)
- added R11: 15, Resistor_SMD:R_1206_3216Metric, F.Cu at (88.9, 100.8)
- added R12: 0.47, Resistor_SMD:R_0805_2012Metric, F.Cu at (52.1, 103.0)
- added R13: 0.47, Resistor_SMD:R_0805_2012Metric, F.Cu at (52.1, 105.9)
- added R14: 0.47, Resistor_SMD:R_0805_2012Metric, F.Cu at (52.1, 108.9)
- added R15: 0.47, Resistor_SMD:R_0805_2012Metric, F.Cu at (52.1, 111.8)
- added R16: 47, Resistor_SMD:R_0603_1608Metric, B.Cu at (99.5, 113.9)
- added R17: 47, Resistor_SMD:R_0603_1608Metric, B.Cu at (99.5, 112.3)
- added R18: 15, Resistor_SMD:R_1206_3216Metric, F.Cu at (88.8, 95.8)
- added R19: 15, Resistor_SMD:R_1206_3216Metric, F.Cu at (88.8, 90.9)
- added R20: 15, Resistor_SMD:R_1206_3216Metric, F.Cu at (88.8, 85.7)
- added R21: 15, Resistor_SMD:R_1206_3216Metric, F.Cu at (88.8, 80.9)
- added R22: 47, Resistor_SMD:R_0603_1608Metric, B.Cu at (95.9, 90.4)
- added R23: 47, Resistor_SMD:R_0603_1608Metric, B.Cu at (95.9, 88.7)
- added R24: 2R2, Resistor_SMD:R_0603_1608Metric, F.Cu at (59.9, 97.8)
- added R25: 1R, Resistor_SMD:R_0805_2012Metric, F.Cu at (52.1, 114.8)
- added R26: 2R2, Resistor_SMD:R_0603_1608Metric, F.Cu at (59.9, 100.3)
- added R27: 4k7, Resistor_SMD:R_0603_1608Metric, F.Cu at (63.9, 85.2)
- added R28: 22k, Resistor_SMD:R_0603_1608Metric, F.Cu at (63.9, 87.7)
- added R29: 22k, Resistor_SMD:R_0603_1608Metric, F.Cu at (63.9, 90.2)
- added R30: 10k, Resistor_SMD:R_0603_1608Metric, F.Cu at (63.9, 92.7)
- added R31: 10k, Resistor_SMD:R_0603_1608Metric, F.Cu at (63.9, 95.2)
- added R32: 4k7, Resistor_SMD:R_0603_1608Metric_Pad0.98x0.95mm_HandSolder, F.Cu at (56.4, 114.2)
- added R33: 4k7, Resistor_SMD:R_0603_1608Metric_Pad0.98x0.95mm_HandSolder, F.Cu at (56.4, 116.7)
- added R6: 0.075, Resistor_SMD:R_1206_3216Metric, B.Cu at (91.1, 88.1)
- added R7: 0.075, Resistor_SMD:R_1206_3216Metric, B.Cu at (91.2, 108.2)
- added R8: 15, Resistor_SMD:R_1206_3216Metric, F.Cu at (88.9, 115.6)
- added R9: 15, Resistor_SMD:R_1206_3216Metric, F.Cu at (88.9, 110.7)
- added U5: AS5047P-ATSM, AS5047P_ATSM:AS5047P_ATSM, B.Cu at (100.0, 100.0)
- moved R5 7.75 mm to (119.8, 98.0), turned to 90 degrees
- moved U4 7.72 mm to (106.9, 100.0), turned to 90 degrees
- moved R4 7.65 mm to (115.2, 98.1), turned to -90 degrees
- moved C8 7.03 mm to (116.7, 98.1), turned to 90 degrees
- moved C9 6.95 mm to (118.3, 98.1), turned to 90 degrees
- moved J1 0.70 mm to (71.7, 103.1)
Connections:
- J1 pad 1: unconnected-(J1-Pin_1-Pad1) -> Coil_B1
- J1 pad 2: unconnected-(J1-Pin_2-Pad2) -> Coil_B2
- J1 pad 3: unconnected-(J1-Pin_3-Pad3) -> Coil_A1
- J1 pad 4: unconnected-(J1-Pin_4-Pad4) -> Coil_A2
- J3 pad 1: unconnected-(J3-Pin_1-Pad1) -> GND
- J3 pad 2: unconnected-(J3-Pin_2-Pad2) -> /IN0/HOME
- J3 pad 3: unconnected-(J3-Pin_3-Pad3) -> /IN1/ENC_A
- J3 pad 4: unconnected-(J3-Pin_4-Pad4) -> /IN2/ENC_B
- J3 pad 5: unconnected-(J3-Pin_5-Pad5) -> /STOP_L/STEP
- J3 pad 6: unconnected-(J3-Pin_6-Pad6) -> /STOP_R/DIR
- J3 pad 7: unconnected-(J3-Pin_7-Pad7) -> /ISO_COM
- J3 pad 8: unconnected-(J3-Pin_8-Pad8) -> /OUT0
- J4 pad 1: unconnected-(J4-Pin_1-Pad1) -> GND
- J4 pad 2: unconnected-(J4-Pin_2-Pad2) -> Vm
- J4 pad 3: unconnected-(J4-Pin_3-Pad3) -> Vm
- J4 pad 4: unconnected-(J4-Pin_4-Pad4) -> /Vlogic
- U2 pad 10: unconnected-(U2-PA0-Pad10) -> DIAG0
- U2 pad 11: unconnected-(U2-PA1-Pad11) -> DIAG1
- U2 pad 12: unconnected-(U2-PA2-Pad12) -> DRV_ENN
- U2 pad 14: unconnected-(U2-PA4-Pad14) -> CSN
- U2 pad 15: unconnected-(U2-PA5-Pad15) -> SCK
- U2 pad 16: unconnected-(U2-PA6-Pad16) -> SPI_MISO
- U2 pad 17: PA7 -> SPI_MOSI
- U2 pad 22: PB11 -> unconnected-(U2-PB11-Pad22)
- U2 pad 25: PB12 -> SPI2_NSS
- U2 pad 26: PB13 -> SPI2_SCK
- U2 pad 27: unconnected-(U2-PB14-Pad27) -> SPI2_MISO
- U2 pad 28: unconnected-(U2-PB15-Pad28) -> SPI2_MOSI
- U4 pad 1: unconnected-(U4-HB1-Pad1) -> HB1
- U4 pad 10: unconnected-(U4-SRBL-Pad10) -> SRBL
- U4 pad 11: unconnected-(U4-TST_MODE-Pad11) -> GND
- U4 pad 12: unconnected-(U4-CLK-Pad12) -> GND
- U4 pad 13: unconnected-(U4-CSN_CFG3-Pad13) -> CSN
- U4 pad 14: unconnected-(U4-SCK_CFG2-Pad14) -> SCK
- U4 pad 15: unconnected-(U4-SDI_CFG1-Pad15) -> SPI_MOSI
- U4 pad 16: unconnected-(U4-SDO_CFG0-Pad16) -> SPI_MISO
- U4 pad 17: unconnected-(U4-REFL_STEP-Pad17) -> REFL
- U4 pad 18: unconnected-(U4-REFR_DIR-Pad18) -> REFR
- U4 pad 19: unconnected-(U4-GNDD-Pad19) -> GND
- U4 pad 2: unconnected-(U4-CB1-Pad2) -> CB1
- U4 pad 20: unconnected-(U4-VCC_IO-Pad20) -> VCC_IO
- U4 pad 21: unconnected-(U4-SD_MODE-Pad21) -> GND
- U4 pad 22: unconnected-(U4-SPI_MODE-Pad22) -> VCC_IO
- U4 pad 23: unconnected-(U4-ENCB_DCEN_CFG4-Pad23) -> ENC_B_channel
- U4 pad 24: unconnected-(U4-ENCA_DCIN_CFG5-Pad24) -> ENC_A_channel
- U4 pad 25: unconnected-(U4-ENCN_DCO_CFG6-Pad25) -> ENC_N_channel_(pull_to_VCC_IO_if_not_used_for_encoder)
- U4 pad 26: unconnected-(U4-DIAG0_SWN-Pad26) -> DIAG0
- U4 pad 27: unconnected-(U4-DIAG1_SWP-Pad27) -> DIAG1
- U4 pad 28: unconnected-(U4-DRV_ENN-Pad28) -> DRV_ENN
- U4 pad 29: unconnected-(U4-VCC-Pad29) -> Net-(U4-VCC)
- U4 pad 3: unconnected-(U4-12VOUT-Pad3) -> Net-(U4-12VOUT)
- U4 pad 30: unconnected-(U4-GNDD-Pad30) -> GND
- U4 pad 31: unconnected-(U4-CPO-Pad31) -> CPO
- U4 pad 32: unconnected-(U4-CPI-Pad32) -> CPI
- U4 pad 33: unconnected-(U4-VS-Pad33) -> VS
- U4 pad 34: unconnected-(U4-VCP-Pad34) -> VCP
- U4 pad 35: unconnected-(U4-CA2-Pad35) -> CA2
- U4 pad 36: unconnected-(U4-HA2-Pad36) -> HA2
- U4 pad 37: unconnected-(U4-BMA2-Pad37) -> BMA2
- U4 pad 38: unconnected-(U4-LA2-Pad38) -> LA2
- U4 pad 39: unconnected-(U4-LA1-Pad39) -> LA1
- U4 pad 4: unconnected-(U4-VSA-Pad4) -> VS
- U4 pad 40: unconnected-(U4-BMA1-Pad40) -> BMA1
- U4 pad 41: unconnected-(U4-HA1-Pad41) -> HA1
- U4 pad 42: unconnected-(U4-CA1-Pad42) -> CA1
- U4 pad 43: unconnected-(U4-CB2-Pad43) -> CB2
- U4 pad 44: unconnected-(U4-HB2-Pad44) -> HB2
- U4 pad 45: unconnected-(U4-BMB2-Pad45) -> BMB2
- U4 pad 46: unconnected-(U4-LB2-Pad46) -> LB2
- U4 pad 47: unconnected-(U4-LB1-Pad47) -> LB1
- U4 pad 48: unconnected-(U4-BMB1-Pad48) -> BMB1
- U4 pad 49: unconnected-(U4-GNDD/GNDP-Pad49) -> GND
- U4 pad 5: unconnected-(U4-5VOUT-Pad5) -> 5VOUT
- U4 pad 6: unconnected-(U4-GNDA-Pad6) -> GND
- U4 pad 7: unconnected-(U4-SRAL-Pad7) -> SRAL
- U4 pad 8: unconnected-(U4-SRAH-Pad8) -> SRAH
- U4 pad 9: unconnected-(U4-SRBH-Pad9) -> SRBH
Routing:
- net Coil_B1: track 0.00 -> 97.8 mm
- net Coil_B2: track 0.00 -> 92.7 mm
- net Coil_A1: track 0.00 -> 67.9 mm
- net SRAL: track 0.00 -> 38.6 mm, vias 0 -> 3
- net SRAH: track 0.00 -> 36.8 mm, vias 0 -> 3
- net Coil_A2: track 0.00 -> 33.4 mm
- net LA2: track 0.00 -> 26.7 mm, vias 0 -> 2
- net HA2: track 0.00 -> 20.9 mm
- net HB1: track 0.00 -> 20.2 mm
- net SRBL: track 0.00 -> 20.1 mm, vias 0 -> 1
- net SRBH: track 0.00 -> 18.2 mm, vias 0 -> 1
- net LB1: track 0.00 -> 17.1 mm
- net LA1: track 0.00 -> 16.2 mm
- net HB2: track 0.00 -> 15.7 mm
- net HA1: track 0.00 -> 13.8 mm
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- added copper zone on B.Cu, net GND
- added copper zone on F.Cu, net GND
- added copper zone on In1.Cu, net GND
- added copper zone on In2.Cu, net Vm
Other:
- copper layers 2 -> 4

Commit message: not finished
Parts:
- removed R32, R33: 4k7, Resistor_SMD:R_0603_1608Metric_Pad0.98x0.95mm_HandSolder
- R12, R13, R14, R15: footprint Resistor_SMD:R_0805_2012Metric -> Resistor_SMD:R_0603_1608Metric
- moved R25 59.2 mm to (106.3, 91.0), turned to -90 degrees
- moved C30 48.1 mm to (103.8, 92.0)
- moved C31 48.0 mm to (103.8, 93.5), turned to 180 degrees
- moved R12 4.38 mm to (50.9, 107.2)
- moved R13 3.95 mm to (50.9, 109.7)
- moved R14 3.53 mm to (50.9, 112.2)
- moved R15 3.12 mm to (50.9, 114.8)
Connections:
- Q1 pad 13: Coil_B1 -> (no net)
- Q1 pad 14: Vm -> (no net)
- Q2 pad 13: Coil_B2 -> (no net)
- Q2 pad 14: Vm -> (no net)
- Q3 pad 13: Coil_A1 -> (no net)
- Q3 pad 14: Vm -> (no net)
- Q4 pad 13: Coil_A2 -> (no net)
- Q4 pad 14: Vm -> (no net)
Routing:
- net VS: track 0.00 -> 6.74 mm
- net VCP: track 0.00 -> 4.05 mm
- net Vm: track 0.00 -> 1.73 mm, vias 60 -> 61
- net HA2: track 20.9 -> 20.1 mm

Commit message: not_finished
Parts:
- removed D4, D5, D6, D7: schotty diode, Diode_SMD:D_MicroSMP_AK
- removed R12, R13, R14, R15: 0.47, Resistor_SMD:R_0603_1608Metric
- C18: moved to B.Cu
- moved C29 53.8 mm to (109.0, 93.6)
- moved C26 52.9 mm to (104.2, 108.5), turned to -90 degrees
- moved C13 51.2 mm to (95.1, 98.0), turned to 180 degrees
- moved C15 50.9 mm to (103.1, 93.8), turned to 180 degrees
- moved R24 50.4 mm to (110.0, 92.1), turned to 180 degrees
- moved C12 48.9 mm to (95.1, 100.0), turned to 180 degrees
- moved C17 46.9 mm to (85.6, 120.3), turned to -90 degrees
- moved C27 44.6 mm to (105.9, 108.3), turned to -90 degrees
- moved C14 44.5 mm to (101.0, 104.3), turned to 180 degrees
- moved C28 41.0 mm to (102.4, 108.2), turned to -90 degrees
- moved C21 39.3 mm to (90.3, 76.5), turned to 90 degrees
- moved C19 36.5 mm to (87.9, 98.6)
- moved C20 34.5 mm to (82.2, 79.0), turned to 90 degrees
- moved C18 30.5 mm to (74.8, 110.3), turned to -90 degrees
- moved R28 10.7 mm to (53.7, 84.3)
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Connections:
- C17 pad 1: Coil_B1 -> BMB1
- C18 pad 1: Coil_B2 -> BMB2
- C19 pad 1: Coil_A1 -> BMA1
- C20 pad 1: Coil_A2 -> BMA2
- J1 pad 1: Coil_B1 -> BMB1
- J1 pad 2: Coil_B2 -> BMB2
- J1 pad 3: Coil_A1 -> BMA1
- J1 pad 4: Coil_A2 -> BMA2
- Q1 pad 1: Coil_B1 -> BMB1
- Q1 pad 11: Coil_B1 -> BMB1
- Q1 pad 12: Coil_B1 -> BMB1
- Q1 pad 5: Coil_B1 -> BMB1
- Q1 pad 6: Coil_B1 -> BMB1
- Q2 pad 1: Coil_B2 -> BMB2
- Q2 pad 11: Coil_B2 -> BMB2
- Q2 pad 12: Coil_B2 -> BMB2
- Q2 pad 5: Coil_B2 -> BMB2
- Q2 pad 6: Coil_B2 -> BMB2
- Q3 pad 1: Coil_A1 -> BMA1
- Q3 pad 11: Coil_A1 -> BMA1
- Q3 pad 12: Coil_A1 -> BMA1
- Q3 pad 5: Coil_A1 -> BMA1
- Q3 pad 6: Coil_A1 -> BMA1
- Q4 pad 1: Coil_A2 -> BMA2
- Q4 pad 11: Coil_A2 -> BMA2
- Q4 pad 12: Coil_A2 -> BMA2
- Q4 pad 5: Coil_A2 -> BMA2
- Q4 pad 6: Coil_A2 -> BMA2
Routing:
- net BMB1: track 0.00 -> 119.6 mm
- net BMB2: track 0.00 -> 108.0 mm, vias 0 -> 1
- net Coil_B1: track 97.8 -> 0.00 mm
- net Coil_B2: track 92.7 -> 0.00 mm
- net BMA1: track 0.00 -> 92.6 mm, vias 0 -> 2
- net Coil_A1: track 67.9 -> 0.00 mm
- net BMA2: track 0.00 -> 58.9 mm
- net Coil_A2: track 33.4 -> 0.00 mm
- net GND: track 0.00 -> 10.2 mm, vias 55 -> 63
- net CA1: track 0.00 -> 6.76 mm
- net CB2: track 0.00 -> 6.70 mm
- net VS: track 6.74 -> 12.7 mm
- net Net-(U4-12VOUT): track 0.00 -> 4.62 mm
- net Net-(U4-VCC): track 0.00 -> 4.38 mm
- net CB1: track 0.00 -> 4.34 mm
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
Commit message: not finished
Parts:
- removed C34, C35: 1n, 100V, Capacitor_SMD:C_0603_1608Metric
- removed R28, R29: 22k, Resistor_SMD:R_0603_1608Metric
- removed R30, R31: 10k, Resistor_SMD:R_0603_1608Metric
- removed R4: 4k7, Resistor_SMD:R_0603_1608Metric_Pad0.98x0.95mm_HandSolder
- added C37: 0.1u, Capacitor_SMD:C_0603_1608Metric_Pad1.08x0.95mm_HandSolder, F.Cu at (120.9, 118.1)
- added C38: 0.1u, Capacitor_SMD:C_0603_1608Metric_Pad1.08x0.95mm_HandSolder, F.Cu at (105.8, 115.8)
- added C39: 1u, Capacitor_SMD:C_0603_1608Metric, B.Cu at (95.5, 99.1)
- added R34: 4k7, Resistor_SMD:R_0603_1608Metric_Pad0.98x0.95mm_HandSolder, F.Cu at (104.2, 118.8)
- added R35: 4k7, Resistor_SMD:R_0603_1608Metric_Pad0.98x0.95mm_HandSolder, F.Cu at (104.2, 117.3)
- C36, R26: moved to B.Cu
- moved C23 66.1 mm to (105.8, 84.0)
- moved C22 60.5 mm to (100.1, 84.0), turned to 180 degrees
- moved C33 57.3 mm to (113.0, 98.5), turned to 90 degrees
- moved C24 56.5 mm to (93.4, 119.6)
- moved R26 54.0 mm to (113.8, 99.3), turned to 180 degrees
- moved C32 50.8 mm to (106.7, 93.2)
- moved R27 47.3 mm to (111.9, 95.1), turned to 180 degrees
- moved C36 44.0 mm to (98.2, 96.3)
- moved J7 43.7 mm to (118.2, 123.1), turned to -90 degrees
- moved R1 39.7 mm to (114.5, 85.7), turned to 90 degrees
- moved C4 39.1 mm to (111.2, 125.7)
- moved D1 32.6 mm to (115.5, 88.2), turned to 180 degrees
- moved D3 25.1 mm to (123.7, 115.9), turned to 0 degrees
- moved D2 24.4 mm to (123.7, 117.6), turned to 0 degrees
- moved R2 17.3 mm to (127.1, 117.5), turned to 0 degrees
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Connections:
- C1 pad 1: 12-24V -> 12-36V
- C21 pad 1: Vm -> 12-36V
- C22 pad 1: Vm -> 12-36V
- C23 pad 1: Vm -> 12-36V
- C24 pad 1: Vm -> 12-36V
- J3 pad 2: /IN0/HOME -> Out_1
- J3 pad 3: /IN1/ENC_A -> Out_2
- J3 pad 6: /STOP_R/DIR -> GND
- J3 pad 7: /ISO_COM -> 5VOUT
- J3 pad 8: /OUT0 -> 5VOUT
- J4 pad 2: Vm -> 12-36V
- J4 pad 3: Vm -> 12-36V
- Q1 pad 10: Vm -> 12-36V
- Q1 pad 7: Vm -> 12-36V
- Q1 pad 8: Vm -> 12-36V
- Q1 pad 9: Vm -> 12-36V
- Q2 pad 10: Vm -> 12-36V
- Q2 pad 7: Vm -> 12-36V
- Q2 pad 8: Vm -> 12-36V
- Q2 pad 9: Vm -> 12-36V
- Q3 pad 10: Vm -> 12-36V
- Q3 pad 7: Vm -> 12-36V
- Q3 pad 8: Vm -> 12-36V
- Q3 pad 9: Vm -> 12-36V
- Q4 pad 10: Vm -> 12-36V
- Q4 pad 7: Vm -> 12-36V
- Q4 pad 8: Vm -> 12-36V
- Q4 pad 9: Vm -> 12-36V
- R1 pad 2: 12-24V -> 12-36V
- R25 pad 1: Vm -> 12-36V
- U1 pad 3: 12-24V -> 12-36V
- U1 pad 4: 12-24V -> 12-36V
- U2 pad 10: DIAG0 -> Net-(U2-PA0)
- U2 pad 11: DIAG1 -> Net-(U2-PA1)
- U2 pad 39: unconnected-(U2-PB3-Pad39) -> Out_1
- U2 pad 40: unconnected-(U2-PB4-Pad40) -> Out_2
- U3 pad 5: CAN_FAULT -> unconnected-(U3-FAULT-Pad5)
Routing:
- net +3V3: track 0.00 -> 131.6 mm, vias 0 -> 4
- net 5VOUT: track 3.25 -> 71.2 mm, vias 0 -> 4
- net GND: track 10.2 -> 48.3 mm, vias 63 -> 93
- net VS: track 12.7 -> 42.2 mm, vias 0 -> 2
- net SPI2_MISO: track 0.00 -> 27.8 mm, vias 0 -> 1
- net SPI2_MOSI: track 0.00 -> 27.7 mm, vias 0 -> 1
- net /TXD: track 0.00 -> 27.5 mm, vias 0 -> 2
- net SPI2_NSS: track 0.00 -> 27.0 mm, vias 0 -> 1
- net DRV_ENN: track 0.00 -> 25.2 mm
- net Out_1: track 0.00 -> 24.8 mm
- net SPI2_SCK: track 0.00 -> 24.4 mm, vias 0 -> 1
- net Out_2: track 0.00 -> 23.7 mm, vias 0 -> 2
- net /NRST: track 0.00 -> 23.6 mm, vias 0 -> 3
- net /RXD: track 0.00 -> 18.7 mm, vias 0 -> 2
- net CSN: track 0.00 -> 15.5 mm, vias 0 -> 2
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- added copper zone on B.Cu, net (none)
- added copper zone on In2.Cu, net 12-36V
- removed copper zone on In2.Cu, net Vm

Commit message: not finished
Parts:
- added C40: 0.1u, Capacitor_SMD:C_0603_1608Metric_Pad1.08x0.95mm_HandSolder, B.Cu at (123.3, 89.4)
- added C41: 4.7u, Capacitor_SMD:C_0603_1608Metric_Pad1.08x0.95mm_HandSolder, B.Cu at (124.7, 89.4)
- added C42: 0.1u, Capacitor_SMD:C_0603_1608Metric_Pad1.08x0.95mm_HandSolder, B.Cu at (119.0, 90.3)
- added C43: 0.1u, Capacitor_SMD:C_0603_1608Metric_Pad1.08x0.95mm_HandSolder, B.Cu at (119.1, 88.8)
- added D8: SP0503BAHT, Package_TO_SOT_SMD:SOT-143, B.Cu at (123.2, 85.4)
- added J5: USB_B_Micro, Connector_USB:USB_Micro-B_Molex-105133-0031, F.Cu at (127.8, 87.5)
- added R36: 4K7, Resistor_SMD:R_0603_1608Metric, F.Cu at (132.5, 72.6)
- added R37: 4K7, Resistor_SMD:R_0603_1608Metric, F.Cu at (132.5, 75.1)
- added R38: 4K7, Resistor_SMD:R_0603_1608Metric, F.Cu at (132.5, 77.6)
- added R39: 1k, Resistor_SMD:R_0603_1608Metric, F.Cu at (127.3, 92.9)
- added R40: 22.1k, Resistor_SMD:R_0603_1608Metric, B.Cu at (125.3, 92.2)
- added R41: 47.5, Resistor_SMD:R_0603_1608Metric, B.Cu at (128.3, 92.2)
- added U6: 24LC02, Housings_SOIC:SOIC-8_3.9x4.9mm_Pitch1.27mm, F.Cu at (126.1, 74.4)
- added U7: CP2102N-Axx-xQFN24, Package_DFN_QFN:QFN-24-1EP_4x4mm_P0.5mm_EP2.6x2.6mm, B.Cu at (121.1, 93.7)
- moved C8 4.85 mm to (116.0, 94.3)
- moved C9 4.85 mm to (117.5, 94.4)
- moved R5 4.80 mm to (114.5, 94.3)
- moved C3 3.57 mm to (121.2, 86.2), turned to 180 degrees
- moved C1 2.39 mm to (116.9, 82.4)
- moved D1 2.39 mm to (116.0, 85.9)
- moved R1 2.39 mm to (114.9, 83.3)
- moved U1 2.39 mm to (120.9, 83.2)
Routing:
- net +3V3: track 131.6 -> 157.2 mm, vias 4 -> 6
- net Net-(J5-VBUS): track 0.00 -> 17.5 mm, vias 0 -> 1
- net /D-: track 0.00 -> 15.2 mm, vias 0 -> 1
- net /D+: track 0.00 -> 13.5 mm, vias 0 -> 1
- net GND: track 48.3 -> 54.5 mm, vias 93 -> 100
- net Net-(U7-VBUS): track 0.00 -> 5.04 mm
- net Net-(U7-~{RST}): track 0.00 -> 4.19 mm, vias 0 -> 1
- net /TXD: track 27.5 -> 29.3 mm
- net Net-(D1-K): track 3.69 -> 3.16 mm
