File: TMCM_1260_alternative/TMCM_1260_alternative.kicad_pcb (KiCad board)
At the start: 4 copper layers, 60 x 60 mm, 93 parts, among them J1 Motor, J2 CAN, J3 I/O, J4 Power, J5 USB_B_Micro, J7 Conn_01x05, Q1 NVMFD5C650NLT1G, Q2 NVMFD5C650NLT1G, Q3 NVMFD5C650NLT1G, Q4 NVMFD5C650NLT1G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

Commit message: not finished
Parts:
- added C44: 0.1u, Capacitor_SMD:C_0603_1608Metric_Pad1.08x0.95mm_HandSolder, B.Cu at (117.5, 96.8)
- R36, R37, R38, U6: moved to B.Cu
- moved R36 33.2 mm to (122.8, 104.4), turned to 90 degrees
- moved R37 30.4 mm to (124.3, 104.4), turned to 90 degrees
- moved R38 27.6 mm to (125.7, 104.4), turned to 90 degrees
- moved U6 25.5 mm to (122.7, 99.7), turned to 180 degrees
- moved J7 0.65 mm to (117.6, 122.9)
Routing:
- net +3V3: track 157.2 -> 165.5 mm, vias 6 -> 7
- net /PC8: track 0.00 -> 8.10 mm
- net /PB8: track 0.00 -> 5.62 mm
- net /PB9: track 0.00 -> 3.98 mm
- net /NRST: track 23.6 -> 25.9 mm

Commit message: not finished
Connections:
- R36 pad 2: /PB9 -> PB0
- R37 pad 2: /PB8 -> PB1
- R38 pad 2: /PC8 -> PB2
- U2 pad 18: unconnected-(U2-PB0-Pad18) -> PB0
- U2 pad 19: unconnected-(U2-PB1-Pad19) -> PB1
- U2 pad 20: unconnected-(U2-PB2-Pad20) -> PB2
- U2 pad 21: unconnected-(U2-PB10-Pad21) -> ?????
- U2 pad 46: unconnected-(U2-PB9-Pad46) -> ????????
- U6 pad 5: /PB9 -> PB0
- U6 pad 6: /PB8 -> PB1
- U6 pad 7: /PC8 -> PB2
Routing:
- net PB2: track 0.00 -> 8.10 mm
- net /PC8: track 8.10 -> 0.00 mm
- net PB1: track 0.00 -> 5.62 mm
- net /PB8: track 5.62 -> 0.00 mm
- net PB0: track 0.00 -> 3.98 mm
- net /PB9: track 3.98 -> 0.00 mm

Commit message: finished
Parts:
- removed C44: 0.1u, Capacitor_SMD:C_0603_1608Metric_Pad1.08x0.95mm_HandSolder
- removed R36, R37, R38: 4K7, Resistor_SMD:R_0603_1608Metric
- removed U6: 24LC02, Housings_SOIC:SOIC-8_3.9x4.9mm_Pitch1.27mm
- added REF**: MountingHole_3.2mm_M3, MountingHole:MountingHole_3.2mm_M3, F.Cu at (116.3, 126.7)
- added REF**: MountingHole_3.2mm_M3, MountingHole:MountingHole_3.2mm_M3, F.Cu at (83.7, 73.3)
- added REF**: MountingHole_3.2mm_M3, MountingHole:MountingHole_3.2mm_M3, F.Cu at (84.0, 125.4)
- added REF**: MountingHole_3.2mm_M3, MountingHole:MountingHole_3.2mm_M3, F.Cu at (116.0, 74.6)
Connections:
- Q1 pad 13: (no net) -> BMB1
- Q1 pad 14: (no net) -> 12-36V
- Q2 pad 13: (no net) -> BMB2
- Q2 pad 14: (no net) -> 12-36V
- Q3 pad 13: (no net) -> BMA1
- Q3 pad 14: (no net) -> 12-36V
- Q4 pad 13: (no net) -> BMA2
- Q4 pad 14: (no net) -> 12-36V
- U1 pad PAD: (no net) -> GND
- U2 pad 21: ????? -> unconnected-(U2-PB10-Pad21)
- U2 pad 30: S_MODE -> UART_TX
- U2 pad 31: CAN_FAULT -> UART_RX
- U2 pad 46: ???????? -> unconnected-(U2-PB9-Pad46)
- U7 pad 20: ???????? -> UART_TX
- U7 pad 21: ????? -> UART_RX
Routing:
- net UART_TX: track 0.00 -> 34.8 mm, vias 0 -> 1
- net UART_RX: track 0.00 -> 31.3 mm, vias 0 -> 1
- net +3V3: track 165.5 -> 157.3 mm, vias 7 -> 6
- net PB2: track 8.10 -> 0.00 mm
- net PB1: track 5.62 -> 0.00 mm
- net PB0: track 3.98 -> 0.00 mm
- net BMB1: track 119.6 -> 116.7 mm
- net BMA1: track 92.6 -> 90.8 mm
- net 5VOUT: track 71.2 -> 73.0 mm, vias 4 -> 3
- net LB2: track 16.0 -> 14.4 mm
- net /NRST: track 25.9 -> 24.7 mm
- net SPI2_MOSI: track 27.7 -> 28.9 mm
- net GND: track 54.5 -> 55.4 mm, vias 100 -> 125
- net VS: track 42.2 -> 43.1 mm
- net BMB2: track 119.3 -> 118.5 mm
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- removed copper zone on B.Cu, net (none)
