File: TMCM_1260_alternative/TMCM_1260_alternative.kicad_sch (KiCad schematic)
At the start: 66 parts, among them J1 Motor, J2 CAN, J3 I/O, J4 Power, J7 Conn_01x05, Q1 NVMFD5C650NLT1G, Q2 NVMFD5C650NLT1G, Q3 NVMFD5C650NLT1G, Q4 NVMFD5C650NLT1G, U1 LMZM23600V3SILR, U2 STM32F091CCTx, U3 TCAN337, U4 TMC5160A-TA-T, Y1 Crystal_Small

Commit message: not finished
Parts:
- added C25: 2n2, symbol Device:C_Small
- added R22, R23: 47, symbol Device:R_Small
Connections:
- net DRAIN_2 is gone; now on net Coil_B1: Q1.11 (D2_3), Q1.12 (D2_4), Q1.5 (D2_1), Q1.6 (D2_2)
- net DRAIN_4 is gone; now on net Coil_B2: Q2.11 (D2_3), Q2.12 (D2_4), Q2.5 (D2_1), Q2.6 (D2_2)
- net DRAIN_6 is gone; now on net Coil_A1: Q3.11 (D2_3), Q3.12 (D2_4), Q3.5 (D2_1), Q3.6 (D2_2)
- net DRAIN_8 is gone; now on net Coil_A2: Q4.11 (D2_3), Q4.12 (D2_4), Q4.5 (D2_1), Q4.6 (D2_2)
- net CA1: now also C13.1, U4.42 (CA1); no longer C13.2, Q3.1 (S1), Q3.10 (D1_4), Q3.7 (D1_1), Q3.8 (D1_2), Q3.9 (D1_3)
- net CA2: now also C15.1, U4.35 (CA2); no longer C15.2, Q4.1 (S1), Q4.10 (D1_4), Q4.7 (D1_1), Q4.8 (D1_2), Q4.9 (D1_3)
- net CB1: now also U4.2 (CB1); no longer Q1.1 (S1), Q1.10 (D1_4), Q1.7 (D1_1), Q1.8 (D1_2), Q1.9 (D1_3)
- net CB2: now also C12.1, U4.43 (CB2); no longer C12.2, Q2.1 (S1), Q2.10 (D1_4), Q2.7 (D1_1), Q2.8 (D1_2), Q2.9 (D1_3)
- net GND: now also C17.2, C18.2, C19.2, C20.2, D4.2 (A), D5.2 (A), D6.2 (A), D7.2 (A), R17.1, R6.2, R7.2, R23.1
- net BMA2: now reaches R15.1
- net BMA2: now also C15.2, D7.1 (K), U4.37 (BMA2)
- net Coil_A2: now reaches R15.2
- net Coil_A2: now also C20.1, Q4.1 (S1)
- net BMB2: now reaches R13.1
- net BMB2: now also C12.2, D5.1 (K), U4.45 (BMB2)
- net Coil_B2: now reaches R13.2
- net Coil_B2: now also C18.1, Q2.1 (S1)
- net Coil_A1: now reaches C19.1
- net Coil_A1: now also Q3.1 (S1), R14.2
- net at R6.1: now also Q3.3 (S2), Q4.3 (S2), R22.1
- net BMB1: now reaches C14.2
- net BMB1: now also D4.1 (K), R12.1, U4.48 (BMB1); no longer U4.2 (CB1)
- net BMA1: now reaches D6.1 (K)
- net BMA1: now also C13.2, R14.1, U4.40 (BMA1)
- net at Q2.3 (S2): now also Q1.3 (S2), R16.1, R7.1
- net Coil_B1: now reaches C17.1
- net Coil_B1: now also Q1.1 (S1), R12.2
- net SRBH: now reaches C16.1
- net SRBH: now also R16.2, U4.9 (SRBH)
- net SRBL: now reaches C16.2
- net SRBL: now also R17.2, U4.10 (SRBL)
- net SRAL: now reaches U4.7 (SRAL)
- net SRAL: now also C25.2, R23.2
- net SRAH: now reaches U4.8 (SRAH)
- net SRAH: now also C25.1, R22.2
- new net DRAIN_1: Q1.10 (D1_4), Q1.7 (D1_1), Q1.8 (D1_2), Q1.9 (D1_3)
- new net DRAIN_3: Q2.10 (D1_4), Q2.7 (D1_1), Q2.8 (D1_2), Q2.9 (D1_3)
- new net DRAIN_5: Q3.10 (D1_4), Q3.7 (D1_1), Q3.8 (D1_2), Q3.9 (D1_3)
- new net DRAIN_7: Q4.10 (D1_4), Q4.7 (D1_1), Q4.8 (D1_2), Q4.9 (D1_3)
Other:
- moved on the sheet: C12, C13, C14, C15, C16, C17, C18, C19, C20, D4, D5, D6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

Commit message: not finished
Parts:
- added C26: 100n, symbol Device:C_Small
- added C27, C28: 10u, symbol Device:C_Small
- added C29, C30, C33: 470n, symbol Device:C_Small
- added C31: 100n, 16V, symbol Device:C_Small
- added C32: 22n, 100V, symbol Device:C_Small
- added C34: 1n, symbol Device:C_Small
- added C35: 1nf, symbol Device:C_Small
- added R24, R26: 2R2, symbol Device:R_Small
- added R25: 1R, symbol Device:R_Small
- added R27: 4k7, symbol Device:R_Small
- added R28, R29: 22k, symbol Device:R_Small
- added R30, R31: 10k, symbol Device:R_Small
- C22, C23, C24: value 100u per 1 amp coil, w low ESR -> 100u per 1 amp coil, w low ESR, electrolitic
- U4: Manufacturer Part Number (none) -> TMC5160A-TA-T; PN (none) -> TMC5160A-TA-T
Connections:
- net PA7 is gone; now on net SPI_MOSI: U2.17 (PA7)
- net Vm is gone; now on net VSA: C21.1, C22.1, C23.1, C24.1
- net Coil_A1: now also J1.3 (Pin_3)
- net Coil_A2: now also J1.4 (Pin_4)
- net Coil_B1: now also J1.1 (Pin_1)
- net Coil_B2: now also J1.2 (Pin_2)
- net GND: now also J3.1 (Pin_1), J4.1 (Pin_1), U4.11 (TST_MODE), U4.12 (CLK), U4.19 (GNDD), U4.21 (SD_MODE), U4.30 (GNDD), U4.6 (GNDA), C26.2, C27.2, C28.2, C29.2, C30.1, C33.2, C34.1, C35.2
- net DIAG0: now reaches U2.10 (PA0)
- net DIAG0: now also U4.26 (DIAG0_SWN)
- net DIAG1: now reaches U2.11 (PA1)
- net DIAG1: now also U4.27 (DIAG1_SWP)
- net DRV_ENN: now reaches U2.12 (PA2)
- net DRV_ENN: now also U4.28 (DRV_ENN), R27.2
- net CSN_ENCODER: now reaches U2.13 (PA3)
- net CSN: now reaches U2.14 (PA4)
- net CSN: now also U4.13 (CSN_CFG3)
- net SCK: now reaches U2.15 (PA5)
- net SCK: now also U4.14 (SCK_CFG2)
- net SPI_MISO: now reaches U2.16 (PA6)
- net SPI_MISO: now also U4.16 (SDO_CFG0)
- net VSA: now reaches J4.2 (Pin_2)
- net VSA: now also J4.3 (Pin_3), U4.4 (VSA), C26.1, R25.1
- net Vlogic: now reaches J4.4 (Pin_4)
- net IN0/HOME: now reaches J3.2 (Pin_2)
- net IN1/ENC_A: now reaches J3.3 (Pin_3)
- net IN2/ENC_B: now reaches J3.4 (Pin_4)
- net STOP_L/STEP: now reaches J3.5 (Pin_5)
- net STOP_R/DIR: now reaches J3.6 (Pin_6)
- net ISO_COM: now reaches J3.7 (Pin_7)
- net OUT0: now reaches J3.8 (Pin_8)
- net SPI_MOSI: now reaches U4.15 (SDI_CFG1)
- net REFL: now reaches U4.17 (REFL_STEP)
- net REFL: now also C35.1, R29.1
- net REFR: now reaches U4.18 (REFR_DIR)
- net REFR: now also C34.2, R28.2
- net VCC_IO: now reaches U4.20 (VCC_IO)
- net VCC_IO: now also U4.22 (SPI_MODE), C33.1, R26.2, R30.2, R31.1
- net ENC_B_channel: now reaches U4.23 (ENCB_DCEN_CFG4)
- net ENC_A_channel: now reaches U4.24 (ENCA_DCIN_CFG5)
- net ENC_N_channel_(pull_to_VCC_IO_if_not_used_for_encoder): now reaches U4.25 (ENCN_DCO_CFG6)
- net at U4.29 (VCC): now also C29.1, R24.2
- net at U4.3 (12VOUT): now also C28.1
- net CPO: now reaches U4.31 (CPO)
- net CPO: now also C32.2
- net CPI: now reaches U4.32 (CPI)
- net CPI: now also C32.1
- net at U4.33 (VS): now also C30.2, C31.1, R25.2
- net VCP: now reaches U4.34 (VCP)
- net VCP: now also C31.2
- net 5VOUT: now reaches U4.5 (5VOUT)
- net 5VOUT: now also C27.1, R24.1, R26.1, R27.1
- new net reference_switch_left: R28.1, R30.1
- new net reference_switch_right: R29.2, R31.2
- no-connect marks 29 -> 25
Other:
- note added: "NOTES:"
- note added: "Vm - max 36V due to use of internal linear regulators, if >= 48V, then need different suppy for VSA pin not higher than 40V, otherwise heating increase for linear regulators"
- moved on the sheet: C1, C10, C11, C12, C13, C14, C15, C16, C17, C18, C19, C2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

Commit message: not finished
Parts:
- added C36: 100n, Capacitor_SMD:C_0603_1608Metric, symbol Device:C_Small
- added R32, R33: 4k7, Resistor_SMD:R_0603_1608Metric_Pad0.98x0.95mm_HandSolder, symbol Device:R_Small
- added U5: AS5047P-ATSM, AS5047P_ATSM:AS5047P_ATSM, symbol AS5047P_ATSM:AS5047P-ATSM
- C12, C13, C14, C15: Manufacturer Part Number (none) -> HMK212C7474KGHTE
- C16, C25, C26, C29, C30, C31, C33: footprint (none) -> Capacitor_SMD:C_0603_1608Metric
- C17, C18, C19, C20: footprint (none) -> Capacitor_SMD:C_0603_1608Metric; Manufacturer Part Number (none) -> GRM1885C2A102JA01D
- C21: footprint (none) -> Capacitor_SMD:C_0805_2012Metric; Manufacturer Part Number (none) -> C2012X5R2A475K125AC
- C22, C23, C24: value 100u per 1 amp coil, w low ESR, electrolitic -> 330u; footprint (none) -> Capacitor_THT:CP_Radial_D10.0mm_P5.00mm; Manufacturer Part Number (none) -> EEU-FS1J331LB
- C27, C28: footprint (none) -> Capacitor_SMD:C_0805_2012Metric
- C32: footprint (none) -> Capacitor_SMD:C_0603_1608Metric; Manufacturer Part Number (none) -> C0603C223K1RACTU
- C34: value 1n -> 1n, 100V; footprint (none) -> Capacitor_SMD:C_0603_1608Metric; Manufacturer Part Number (none) -> GRM1885C2A102JA01D
- C35: value 1nf -> 1n, 100V; footprint (none) -> Capacitor_SMD:C_0603_1608Metric; Manufacturer Part Number (none) -> GRM1885C2A102JA01D
- D4, D5, D6, D7: value 1A type schotty diode (full/over Vm range) -> schotty diode; footprint (none) -> Diode_SMD:D_MicroSMP_AK; Manufacturer Part Number (none) -> MSS1P6-M3/89A
- R10, R11, R18, R19, R20, R21, R8, R9: Manufacturer Part Number (none) -> RNCP1206FTD15R0
- R12, R13, R14, R15: footprint (none) -> Resistor_SMD:R_0805_2012Metric; Manufacturer Part Number (none) -> ERJ-6DQJR47V
- R16, R17, R22, R23, R24, R26, R27, R28, R29, R30, R31: footprint (none) -> Resistor_SMD:R_0603_1608Metric
- R25: footprint (none) -> Resistor_SMD:R_0805_2012Metric
- R6, R7: value 0.022 -> 0.075; footprint Resistor_SMD:R_2512_6332Metric -> Resistor_SMD:R_1206_3216Metric; Manufacturer Part Number (none) -> ERJ-8BWFR075V; PN TLRP3A30CR022FTE -> ERJ-8BWFR075V
Connections:
- net DRAIN_3 is gone; now on net Vm: Q2.10 (D1_4), Q2.7 (D1_1), Q2.8 (D1_2), Q2.9 (D1_3)
- net DRAIN_5 is gone; now on net Vm: Q3.10 (D1_4), Q3.7 (D1_1), Q3.8 (D1_2), Q3.9 (D1_3)
- net DRAIN_7 is gone; now on net Vm: Q4.10 (D1_4), Q4.7 (D1_1), Q4.8 (D1_2), Q4.9 (D1_3)
- net +3V3: now also C36.2, R32.2, R33.2, U5.11 (VDD), U5.12 (VDD3V)
- net DIAG0: now also R33.1
- net DIAG1: now also R32.1
- net GND: now also C36.1, U5.13 (GND), U5.5 (TEST)
- net reference_switch_left: now also R29.2, R31.2; no longer R28.1, R30.1
- net reference_switch_right: now also R28.1, R30.1; no longer R29.2, R31.2
- net VS: now reaches C30.2, C31.1, R25.2, U4.33 (VS)
- net VS: now also C26.1, U4.4 (VSA)
- net SPI2_MISO: now reaches U2.27 (PB14)
- net SPI2_MISO: now also U5.3 (MISO)
- net SPI2_MOSI: now reaches U2.28 (PB15)
- net SPI2_MOSI: now also U5.4 (MOSI)
- net CSN_ENCODER: no longer names the net of U2.13 (PA3)
- net DRAIN_1 renamed Vm
- net Vm: now also C21.1, C22.1, C23.1, C24.1, J4.2 (Pin_2), J4.3 (Pin_3), R25.1
- net PB11: no longer names the net of U2.22 (PB11)
- net PB12 renamed SPI2_NSS
- net SPI2_NSS: now also U5.1 (CSn)
- net PB13 renamed SPI2_SCK
- net SPI2_SCK: now also U5.2 (CLK)
- removed net VSA: C21.1, C22.1, C23.1, C24.1, C26.1, J4.2 (Pin_2), J4.3 (Pin_3), R25.1, U4.4 (VSA)
- no-connect marks 25 -> 31
Other:
- note added: "AS5047P-ATSM - SPI MODE:1; TMC5160 - SPI MODE:3;"
- note added: "https://www.digikey.lv/en/products/detail/analog-devices-inc-maxim-integrated/PD57-2-1260-CANOPEN/9381887 Current rating: 2.8 amps for our motors, so no need for high current settings"
- moved on the sheet: C26, C27, C28

Commit message: not finished
Parts:
- R12, R13, R14, R15: footprint Resistor_SMD:R_0805_2012Metric -> Resistor_SMD:R_0603_1608Metric; Manufacturer Part Number ERJ-6DQJR47V -> 73L2R47J
- R32, R33: now not fitted
Changed lines of the file:
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@@
 		(exclude_from_sim no)
 		(in_bom yes)
-		(on_board yes)
-		(dnp no)
+		(on_board no)
+		(dnp yes)
 		(property "Reference" "R33"
 			(at 189.1284 306.07 90)
@@
 	(symbol
 		(lib_id "Device:R_Small")
-		(at 245.11 158.75 90)
+		(at 246.38 95.25 90)
 		(unit 1)
 		(exclude_from_sim no)
@@
 		(dnp no)
 		(fields_autoplaced yes)
-		(property "Reference" "R14"
-			(at 245.11 153.67 90)
+		(property "Reference" "R12"
+			(at 246.38 90.17 90)
 			(effects
 				(font
@@
 		)
 		(property "Value" "0.47"
-			(at 245.11 156.21 90)
+			(at 246.38 92.71 90)
 			(effects
 				(font
@@
 			)
 		)
-		(property "Footprint" "Resistor_SMD:R_0805_2012Metric"
-			(at 245.11 158.75 0)
+		(property "Footprint" "Resistor_SMD:R_0603_1608Metric"
+			(at 246.38 95.25 0)
 			(effects
 				(font
@@
 			)
 		)
-		(property "Datasheet" "https://www.digikey.com/en/products/detail/panasonic-electronic-components/ERJ-6DQJR47V/6004335"
-			(at 245.11 158.75 0)
+		(property "Datasheet" "https://www.digikey.com/en/products/detail/cts-resistor-products/73L2R47J/1543468"
+			(at 246.38 95.25 0)
 			(effects
 				(font
@@
 			)
 		)
-		(property "Description" "RES 0.47 OHM 5% 1/2W 0805"
-			(at 245.11 158.75 0)
+		(property "Description" "RES 0.47 OHM 5% 1/10W 0603"
+			(at 246.38 95.25 0)
 			(effects
 				(font
@@
 			)
 		)
-		(property "Manufacturer Part Number" "ERJ-6DQJR47V"
-			(at 245.11 158.75 0)
+		(property "Manufacturer Part Number" "73L2R47J"
+			(at 246.38 95.25 0)
 			(effects
 				(font
@@
 			(project "TMCM_1260_alternative"
 				(path "/e4fb31fb-ec55-43a1-9d58-e537a4a0024e"
-					(reference "R14")
+					(reference "R12")
 					(unit 1)
 				)
@@
 	)
 	(symbol
-		(lib_id "Device:R_Small")
-		(at 309.88 95.25 90)
-		(unit 1)
-		(exclude_from_sim no)
-		(in_bom yes)
-		(on_board yes)
-		(dnp no)
-		(fields_autoplaced yes)
-		(property "Reference" "R13"
-			(at 309.88 90.17 90)
-			(effects
-				(font
-					(size 1.27 1.27)
-				)
-			)
-		)
-		(property "Value" "0.47"
-			(at 309.88 92.71 90)
-			(effects
-				(font
-					(size 1.27 1.27)
-				)
-			)
-		)
-		(property "Footprint" "Resistor_SMD:R_0805_2012Metric"
-			(at 309.88 95.25 0)
-			(effects
-				(font
-					(size 1.27 1.27)
-				)
-				(hide yes)
-			)
-		)
-		(property "Datasheet" "https://www.digikey.com/en/products/detail/panasonic-electronic-components/ERJ-6DQJR47V/6004335"
-			(at 309.88 95.25 0)
-			(effects
-				(font
-					(size 1.27 1.27)
-				)
-				(hide yes)
-			)
-		)
-		(property "Description" "RES 0.47 OHM 5% 1/2W 0805"
-			(at 309.88 95.25 0)
-			(effects
-				(font
-					(size 1.27 1.27)
-				)
-				(hide yes)
-			)
-		)
-		(property "Manufacturer Part Number" "ERJ-6DQJR47V"
-			(at 309.88 95.25 0)
-			(effects
-				(font
-					(size 1.27 1.27)
-				)
-				(hide yes)
-			)
-		)
-		(pin "1"
-		)
-		(pin "2"
-		)
-		(instances
-			(project "TMCM_1260_alternative"
-				(path "/e4fb31fb-ec55-43a1-9d58-e537a4a0024e"
-					(reference "R13")
-					(unit 1)
-				)
-			)
-		)
-	)
-	(symbol
 		(lib_id "Device:LED")
 		(at 102.87 374.65 0)
@@
 	(symbol
 		(lib_id "Device:R_Small")
+		(at 309.88 95.25 90)
+		(unit 1)
+		(exclude_from_sim no)
+		(in_bom yes)
+		(on_board yes)
+		(dnp no)
+		(fields_autoplaced yes)
+		(property "Reference" "R13"
+			(at 309.88 90.17 90)
+			(effects
+				(font
+					(size 1.27 1.27)
+				)
+			)
+		)
+		(property "Value" "0.47"
+			(at 309.88 92.71 90)
+			(effects
+				(font
+					(size 1.27 1.27)
+				)
+			)
+		)
+		(property "Footprint" "Resistor_SMD:R_0603_1608Metric"
+			(at 309.88 95.25 0)
+			(effects
+				(font
+					(size 1.27 1.27)
+				)
+				(hide yes)
+			)
+		)
+		(property "Datasheet" "https://www.digikey.com/en/products/detail/cts-resistor-products/73L2R47J/1543468"
+			(at 309.88 95.25 0)
+			(effects
+				(font
+					(size 1.27 1.27)
+				)
+				(hide yes)
+			)
+		)
+		(property "Description" "RES 0.47 OHM 5% 1/10W 0603"
+			(at 309.88 95.25 0)
+			(effects
+				(font
+					(size 1.27 1.27)
+				)
+				(hide yes)
+			)
+		)
+		(property "Manufacturer Part Number" "73L2R47J"
+			(at 309.88 95.25 0)
+			(effects
+				(font
+					(size 1.27 1.27)
+				)
+				(hide yes)
+			)
+		)
+		(pin "1"
+		)
+		(pin "2"
+		)
+		(instances
+			(project "TMCM_1260_alternative"
+				(path "/e4fb31fb-ec55-43a1-9d58-e537a4a0024e"
+					(reference "R13")
+					(unit 1)
+				)
+			)
+		)
+	)
+	(symbol
+		(lib_id "Device:R_Small")
 		(at 185.42 383.54 0)
 		(unit 1)
@@
 			)
 		)
-		(property "Footprint" "Resistor_SMD:R_0805_2012Metric"
+		(property "Footprint" "Resistor_SMD:R_0603_1608Metric"
 			(at 308.61 158.75 0)
 			(effects
@@
 			)
 		)
-		(property "Datasheet" "https://www.digikey.com/en/products/detail/panasonic-electronic-components/ERJ-6DQJR47V/6004335"
+		(property "Datasheet" "https://www.digikey.com/en/products/detail/cts-resistor-products/73L2R47J/1543468"
 			(at 308.61 158.75 0)
 			(effects
@@
 			)
 		)
-		(property "Description" "RES 0.47 OHM 5% 1/2W 0805"
+		(property "Description" "RES 0.47 OHM 5% 1/10W 0603"
 			(at 308.61 158.75 0)
 			(effects
@@
 			)
 		)
-		(property "Manufacturer Part Number" "ERJ-6DQJR47V"
+		(property "Manufacturer Part Number" "73L2R47J"
 			(at 308.61 158.75 0)
 			(effects
@@
 	(symbol
 		(lib_id "Device:R_Small")
+		(at 245.11 158.75 90)
+		(unit 1)
+		(exclude_from_sim no)
+		(in_bom yes)
+		(on_board yes)
+		(dnp no)
+		(fields_autoplaced yes)
+		(property "Reference" "R14"
+			(at 245.11 153.67 90)
+			(effects
+				(font
+					(size 1.27 1.27)
+				)
+			)
+		)
+		(property "Value" "0.47"
+			(at 245.11 156.21 90)
+			(effects
+				(font
+					(size 1.27 1.27)
+				)
+			)
+		)
+		(property "Footprint" "Resistor_SMD:R_0603_1608Metric"
+			(at 245.11 158.75 0)
+			(effects
+				(font
+					(size 1.27 1.27)
+				)
+				(hide yes)
+			)
+		)
+		(property "Datasheet" "https://www.digikey.com/en/products/detail/cts-resistor-products/73L2R47J/1543468"
+			(at 245.11 158.75 0)
+			(effects
+				(font
+					(size 1.27 1.27)
+				)
+				(hide yes)
+			)
+		)
+		(property "Description" "RES 0.47 OHM 5% 1/10W 0603"
+			(at 245.11 158.75 0)
+			(effects
+				(font
+					(size 1.27 1.27)
+				)
+				(hide yes)
+			)
+		)
+		(property "Manufacturer Part Number" "73L2R47J"
+			(at 245.11 158.75 0)
+			(effects
+				(font
+					(size 1.27 1.27)
+				)
+				(hide yes)
+			)
+		)
+		(pin "1"
+		)
+		(pin "2"
+		)
+		(instances
+			(project "TMCM_1260_alternative"
+				(path "/e4fb31fb-ec55-43a1-9d58-e537a4a0024e"
+					(reference "R14")
+					(unit 1)
+				)
+			)
+		)
+	)
+	(symbol
+		(lib_id "Device:R_Small")
 		(at 309.88 172.72 90)
 		(unit 1)
@@
 	)
 	(symbol
-		(lib_id "Device:R_Small")
-		(at 246.38 95.25 90)
-		(unit 1)
-		(exclude_from_sim no)
-		(in_bom yes)
-		(on_board yes)
-		(dnp no)
-		(fields_autoplaced yes)
-		(property "Reference" "R12"
-			(at 246.38 90.17 90)
-			(effects
-				(font
-					(size 1.27 1.27)
-				)
-			)
-		)
-		(property "Value" "0.47"
-			(at 246.38 92.71 90)
-			(effects
-				(font
-					(size 1.27 1.27)
-				)
-			)
-		)
-		(property "Footprint" "Resistor_SMD:R_0805_2012Metric"
-			(at 246.38 95.25 0)
-			(effects
-				(font
-					(size 1.27 1.27)
-				)
-				(hide yes)
-			)
-		)
-		(property "Datasheet" "https://www.digikey.com/en/products/detail/panasonic-electronic-components/ERJ-6DQJR47V/6004335"
-			(at 246.38 95.25 0)
-			(effects
-				(font
-					(size 1.27 1.27)
-				)
-				(hide yes)
-			)
-		)
-		(property "Description" "RES 0.47 OHM 5% 1/2W 0805"
-			(at 246.38 95.25 0)
-			(effects
-				(font
-					(size 1.27 1.27)
-				)
-				(hide yes)
-			)
-		)
-		(property "Manufacturer Part Number" "ERJ-6DQJR47V"
-			(at 246.38 95.25 0)
-			(effects
-				(font
-					(size 1.27 1.27)
-				)
-				(hide yes)
-			)
-		)
-		(pin "1"
-		)
-		(pin "2"
-		)
-		(instances
-			(project ""
-				(path "/e4fb31fb-ec55-43a1-9d58-e537a4a0024e"
-					(reference "R12")
-					(unit 1)
-				)
-			)
-		)
-	)
-	(symbol
 		(lib_id "Device:C_Small")
 		(at 297.18 154.94 90)
@@
 		(exclude_from_sim no)
 		(in_bom yes)
-		(on_board yes)
-		(dnp no)
+		(on_board no)
+		(dnp yes)
 		(property "Reference" "R32"
 			(at 191.6684 311.15 90)

Commit message: not_finished
Parts:
- D4, D5, D6, D7, R12, R13, R14, R15: now not fitted
Connections:
- net Coil_A1 is gone; now on net BMA1: C19.1, J1.3 (Pin_3), Q3.1 (S1), Q3.11 (D2_3), Q3.12 (D2_4), Q3.5 (D2_1), Q3.6 (D2_2), R14.2
- net Coil_A2 is gone; now on net BMA2: C20.1, J1.4 (Pin_4), Q4.1 (S1), Q4.11 (D2_3), Q4.12 (D2_4), Q4.5 (D2_1), Q4.6 (D2_2), R15.2
- net Coil_B1 is gone; now on net BMB1: C17.1, J1.1 (Pin_1), Q1.1 (S1), Q1.11 (D2_3), Q1.12 (D2_4), Q1.5 (D2_1), Q1.6 (D2_2), R12.2
- net Coil_B2 is gone; now on net BMB2: C18.1, J1.2 (Pin_2), Q2.1 (S1), Q2.11 (D2_3), Q2.12 (D2_4), Q2.5 (D2_1), Q2.6 (D2_2), R13.2

Commit message: not finished
Parts:
- added C37, C38: 0.1u, Capacitor_SMD:C_0603_1608Metric_Pad1.08x0.95mm_HandSolder, symbol Device:C
- added C39: 1u, Capacitor_SMD:C_0603_1608Metric, symbol Device:C_Small
- added R34, R35: 4k7, Resistor_SMD:R_0603_1608Metric_Pad0.98x0.95mm_HandSolder, symbol Device:R_Small
- C34, C35, R28, R29, R30, R31, R4: now not fitted
Connections:
- net 12-24V is gone; now on net Vm: C1.1, R1.2, U1.3 (VIN), U1.4 (EN)
- net IN0/HOME is gone; now on net Out_1: J3.2 (Pin_2)
- net IN1/ENC_A is gone; now on net Out_2: J3.3 (Pin_3)
- net ISO_COM is gone; now on net 5VOUT: J3.7 (Pin_7)
- net OUT0 is gone; now on net 5VOUT: J3.8 (Pin_8)
- net STOP_R/DIR is gone; now on net GND: J3.6 (Pin_6)
- net +3V3: now also C37.1, C39.2
- net 5VOUT: now also C38.1, R34.2, R35.2
- net CAN_FAULT: no longer U3.5 (FAULT)
- net DIAG0: no longer R33.1, U2.10 (PA0)
- net DIAG1: no longer R32.1, U2.11 (PA1)
- net GND: now also C37.2, C38.2, C39.1
- net Out_1: now reaches U2.39 (PB3)
- net Out_1: now also R35.1
- net Out_2: now reaches U2.40 (PB4)
- net Out_2: now also R34.1
- new net: R33.1, U2.10 (PA0)
- new net: R32.1, U2.11 (PA1)
- no-connect marks 31 -> 30

Commit message: not finished
Parts:
- added C40, C42, C43: 0.1u, Capacitor_SMD:C_0603_1608Metric_Pad1.08x0.95mm_HandSolder, symbol Device:C
- added C41: 4.7u, Capacitor_SMD:C_0603_1608Metric_Pad1.08x0.95mm_HandSolder, symbol Device:C
- added D8: SP0503BAHT, Package_TO_SOT_SMD:SOT-143, symbol Power_Protection:SP0503BAHT
- added J5: USB_B_Micro, Connector_USB:USB_Micro-B_Molex-105133-0031, symbol Connector:USB_B_Micro
- added R36, R37, R38: 4K7, Resistor_SMD:R_0603_1608Metric, symbol Device:R
- added R39: 1k, Resistor_SMD:R_0603_1608Metric, symbol Device:R
- added R40: 22.1k, Resistor_SMD:R_0603_1608Metric, symbol Device:R
- added R41: 47.5, Resistor_SMD:R_0603_1608Metric, symbol Device:R
- added U6: 24LC02, Housings_SOIC:SOIC-8_3.9x4.9mm_Pitch1.27mm, symbol Memory_EEPROM:24LC02
- added U7: CP2102N-Axx-xQFN24, Package_DFN_QFN:QFN-24-1EP_4x4mm_P0.5mm_EP2.6x2.6mm, symbol Interface_USB:CP2102N-Axx-xQFN24
Connections:
- net +3V3: now also C42.1, C43.1, R36.1, R37.1, R38.1, R39.2, U6.8 (VCC), U7.5 (VIO), U7.6 (VDD)
- net GND: now also C40.1, C41.1, C42.2, C43.2, D8.1 (A), J5.5 (GND), J5.6 (Shield), R41.1, U6.1 (A0), U6.2 (A1), U6.3 (A2), U6.4 (GND), U7.2 (GND), U7.25 (GND)
- new net: R39.1, U7.9 (~{RST})
- new net: C40.2, C41.2, D8.4 (K), J5.1 (VBUS), R40.2, U7.7 (VREGIN)
- new net: R40.1, R41.2, U7.8 (VBUS)
- new net ?????: U7.21 (TXD)
- new net ????????: U7.20 (RXD)
- new net D+: D8.2 (K), J5.3 (D+), U7.3 (D+)
- new net D-: D8.3 (K), J5.2 (D-), U7.4 (D-)
- new net PB8: R37.2, U6.6 (SCL)
- new net PB9: R36.2, U6.5 (SDA)
- new net PC8: R38.2, U6.7 (WP)
- no-connect marks 30 -> 31
