File: TMCM_1260_alternative/TMCM_1260_alternative.kicad_sch (KiCad schematic)
At the start: 111 parts, among them J1 Motor, J2 CAN, J3 I/O, J4 Power, J5 USB_B_Micro, J7 Conn_01x05, Q1 NVMFD5C650NLT1G, Q2 NVMFD5C650NLT1G, Q3 NVMFD5C650NLT1G, Q4 NVMFD5C650NLT1G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

Commit message: not finished
Connections:
- net PB8 is gone; now on net PB1: R37.2, U6.6 (SCL)
- net PB9 is gone; now on net PB0: R36.2, U6.5 (SDA)
- net PC8 is gone; now on net PB2: R38.2, U6.7 (WP)
- net ?????: now also U2.21 (PB10)
- net ????????: now also U2.46 (PB9)
- net PB0: now reaches U2.18 (PB0)
- net PB1: now reaches U2.19 (PB1)
- net PB2: now reaches U2.20 (PB2)
- no-connect marks 31 -> 26
Changed lines of the file:
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@@
 	)
 	(no_connect
-		(at 152.4 321.31)
-	)
-	(no_connect
 		(at 196.85 204.47)
 	)
@@
 	)
 	(no_connect
-		(at 152.4 339.09)
-	)
-	(no_connect
 		(at 62.23 40.64)
 	)
@@
 	)
 	(no_connect
-		(at 152.4 316.23)
-	)
-	(no_connect
-		(at 152.4 318.77)
-	)
-	(no_connect
 		(at 156.21 219.71)
 	)
@@
 	)
 	(no_connect
-		(at 152.4 341.63)
-	)
-	(no_connect
 		(at 196.85 217.17)
 	)
@@
 	(wire
 		(pts
+			(xy 149.86 341.63) (xy 152.4 341.63)
+		)
+		(stroke
+			(width 0)
+			(type default)
+		)
+	)
+	(wire
+		(pts
 			(xy 54.61 163.83) (xy 54.61 166.37)
 		)
@@
 	(wire
 		(pts
+			(xy 151.13 321.31) (xy 152.4 321.31)
+		)
+		(stroke
+			(width 0)
+			(type default)
+		)
+	)
+	(wire
+		(pts
 			(xy 190.5 120.65) (xy 191.77 120.65)
 		)
@@
 	(wire
 		(pts
+			(xy 149.86 339.09) (xy 152.4 339.09)
+		)
+		(stroke
+			(width 0)
+			(type default)
+		)
+	)
+	(wire
+		(pts
 			(xy 345.44 120.65) (xy 345.44 118.11)
 		)
@@
 	(wire
 		(pts
+			(xy 151.13 318.77) (xy 152.4 318.77)
+		)
+		(stroke
+			(width 0)
+			(type default)
+		)
+	)
+	(wire
+		(pts
 			(xy 222.25 125.73) (xy 228.6 125.73)
 		)
@@
 	(wire
 		(pts
+			(xy 151.13 316.23) (xy 152.4 316.23)
+		)
+		(stroke
+			(width 0)
+			(type default)
+		)
+	)
+	(wire
+		(pts
 			(xy 312.42 161.29) (xy 304.8 161.29)
 		)
@@
 		)
 	)
-	(label "PB9"
+	(label "PB0"
 		(at 233.68 285.75 0)
 		(effects
@@
 		)
 	)
-	(label "PC8"
+	(label "PB2"
 		(at 254.635 290.83 180)
 		(effects
@@
 		)
 	)
-	(label "PB8"
+	(label "PB1"
 		(at 243.205 288.29 0)
 		(effects
@@
 		)
 	)
+	(global_label "PB2"
+		(shape input)
+		(at 151.13 321.31 180)
+		(fields_autoplaced yes)
+		(effects
+			(font
+				(size 1.27 1.27)
+			)
+			(justify right)
+		)
+		(property "Intersheetrefs" "${INTERSHEET_REFS}"
+			(at 144.3953 321.31 0)
+			(effects
+				(font
+					(size 1.27 1.27)
+				)
+				(justify right)
+				(hide yes)
+			)
+		)
+	)
 	(global_label "PB3"
 		(shape input)
@@
 		)
 	)
+	(global_label "PB0"
+		(shape input)
+		(at 151.13 316.23 180)
+		(fields_autoplaced yes)
+		(effects
+			(font
+				(size 1.27 1.27)
+			)
+			(justify right)
+		)
+		(property "Intersheetrefs" "${INTERSHEET_REFS}"
+			(at 144.3953 316.23 0)
+			(effects
+				(font
+					(size 1.27 1.27)
+				)
+				(justify right)
+				(hide yes)
+			)
+		)
+	)
 	(global_label "BMB2"
 		(shape input)
@@
 		)
 	)
+	(global_label "????????"
+		(shape input)
+		(at 149.86 339.09 180)
+		(fields_autoplaced yes)
+		(effects
+			(font
+				(size 1.27 1.27)
+			)
+			(justify right)
+		)
+		(property "Intersheetrefs" "${INTERSHEET_REFS}"
+			(at 138.166 339.09 0)
+			(effects
+				(font
+					(size 1.27 1.27)
+				)
+				(justify right)
+				(hide yes)
+			)
+		)
+	)
 	(global_label "GNDA"
 		(shape input)
@@
 		)
 	)
+	(global_label "?????"
+		(shape input)
+		(at 149.86 341.63 180)
+		(fields_autoplaced yes)
+		(effects
+			(font
+				(size 1.27 1.27)
+			)
+			(justify right)
+		)
+		(property "Intersheetrefs" "${INTERSHEET_REFS}"
+			(at 141.4318 341.63 0)
+			(effects
+				(font
+					(size 1.27 1.27)
+				)
+				(justify right)
+				(hide yes)
+			)
+		)
+	)
 	(global_label "5VOUT"
 		(shape input)
@@
 				(hide yes)
 			)
+		)
+	)
+	(global_label "PB1"
+		(shape input)
+		(at 151.13 318.77 180)
+		(fields_autoplaced yes)
+		(effects
+			(font
+				(size 1.27 1.27)
+			)
+			(justify right)
+		)
+		(property "Intersheetrefs" "${INTERSHEET_REFS}"
+			(at 144.3953 318.77 0)
+			(effects
+				(font
+					(size 1.27 1.27)
+				)
+				(justify right)
+				(hide yes)
+			)

Commit message: finished
Parts:
- removed C44: 0.1u, Capacitor_SMD:C_0603_1608Metric_Pad1.08x0.95mm_HandSolder, symbol Device:C
- removed R36, R37, R38: 4K7, Resistor_SMD:R_0603_1608Metric, symbol Device:R
- removed U6: 24LC02, Housings_SOIC:SOIC-8_3.9x4.9mm_Pitch1.27mm, symbol Memory_EEPROM:24LC02
- U7: PN (none) -> CP2102N-A02-GQFN24R
Connections:
- net CAN_FAULT: no longer U2.31 (PA10)
- net ?????: no longer names the net of U2.21 (PB10)
- net ?????: no longer U7.21 (TXD)
- net ????????: no longer names the net of U2.46 (PB9)
- net ????????: no longer U7.20 (RXD)
- net S_MODE renamed UART_TX
- net UART_TX: now also U7.20 (RXD)
- new net UART_RX: U2.31 (PA10), U7.21 (TXD)
- no-connect marks 26 -> 28
