File: TMCM_1260_alternative_ver_2/TMCM_1260_alternative_ver_2.kicad_sch (KiCad schematic)
At the start: 106 parts, among them J1 Motor, J2 CAN, J3 I/O, J4 Power, J5 USB_B_Micro, J7 Conn_01x05, Q1 NVMFD5C650NLT1G, Q2 NVMFD5C650NLT1G, Q3 NVMFD5C650NLT1G, Q4 NVMFD5C650NLT1G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

Commit message: iterration 2 upload
Parts:
- added J6: JXD2-0Z10NL, JXD2_0Z10NL:JXD2_0Z10NL, symbol JXD2_0Z10NL:JXD2-0Z10NL
- added U6: STM32H563RGTx, Package_QFP:LQFP-64_10x10mm_P0.5mm, symbol MCU_ST_STM32H5:STM32H563RGTx
- added U8: TMC4361A-LA-T, TMC4361A_LA_T:TMC4361A_LA_T, symbol TMC4361A_LA_T:TMC4361A-LA-T
- added U9: LAN8742A-CZ-TR, LAN8742A_CZ_TR:LAN8742A_CZ_TR, symbol LAN8742A_CZ_TR:LAN8742A-CZ-TR
Connections:
- new net: U6.18 (VSS), U6.31 (VSS), U6.47 (VSS), U6.63 (VSS)
Other:
- note added: "EXTERNAL shield that connects via pins on driver board and fixed with one screw"
- note added: "in stm32 place on driver board"
- note added: "incremental ABI direct connection to TMC4361A-LA-T"
- note added: "will be migrating to STM32H563RGT6"
