File: TMCM_1260_alternative_ver_2/TMCM_1260_alternative_ver_2.kicad_sch (KiCad schematic)
At the start: 110 parts, among them J1 Motor, J2 CAN, J3 I/O, J4 Power, J5 USB_B_Micro, J6 JXD2-0Z10NL, J7 Conn_01x05, Q1 NVMFD5C650NLT1G, Q2 NVMFD5C650NLT1G, Q3 NVMFD5C650NLT1G, Q4 NVMFD5C650NLT1G, U1 LMZM23600V3SILR, U2 STM32F091CCTx, U3 TCAN337, U4 TMC5160A-TA-T, U5 AS5047P-ATSM, U6 STM32H563RGTx, U7 CP2102N-Axx-xQFN24, U8 TMC4361A-LA-T, U9 LAN8742A-CZ-TR, Y1 Crystal_Small

Commit message: upload
Parts:
- removed J6: JXD2-0Z10NL, JXD2_0Z10NL:JXD2_0Z10NL, symbol JXD2_0Z10NL:JXD2-0Z10NL
- added J6: JXD2-0Z10NL, JXD2_0Z10NL:JXD2_0Z10NL, symbol JXD2-0Z10NL:JXD2-0Z10NL

Commit message: tmc4361 added ver_2
Parts:
- removed U2: STM32F091CCTx, Package_QFP:LQFP-48_7x7mm_P0.5mm, symbol MCU_ST_STM32F0:STM32F091CCTx
- removed Y1: Crystal_Small, digikey-footprints:SMD-2_3.2x2.5mm, symbol Device:Crystal_Small
- added C44, C45: 2.2u, Capacitor_SMD:C_0603_1608Metric_Pad1.08x0.95mm_HandSolder, symbol Device:C
- added C46: 4.7u, Capacitor_SMD:C_0603_1608Metric_Pad1.08x0.95mm_HandSolder, symbol Device:C
- added C47, C48: 15p, Capacitor_SMD:C_0603_1608Metric, symbol Device:C
- added C49, C57, C58, C59, C60, C61, C62: 0.1u, Capacitor_SMD:C_0603_1608Metric_Pad1.08x0.95mm_HandSolder, symbol Device:C
- added C50: 470p, Capacitor_SMD:C_0603_1608Metric_Pad1.08x0.95mm_HandSolder, symbol Device:C
- added C51: 1u, Capacitor_SMD:C_0603_1608Metric_Pad1.08x0.95mm_HandSolder, symbol Device:C
- added C52, C53, C54, C56: 10pF, Capacitor_SMD:C_0603_1608Metric_Pad1.08x0.95mm_HandSolder, symbol Device:C
- added C55: 0.022uF, Capacitor_SMD:C_0603_1608Metric_Pad1.08x0.95mm_HandSolder, symbol Device:C
- added R36, R37: 330, Resistor_SMD:R_0603_1608Metric, symbol Device:R_Small
- added R38, R42, R43, R44: 49.9, Resistor_SMD:R_0603_1608Metric, symbol Device:R_Small
- added R45, R46, R47: 100, Resistor_SMD:R_0603_1608Metric, symbol Device:R_Small
- added Y2: 25Mhz, Crystal:Crystal_SMD_2016-4Pin_2.0x1.6mm, symbol Device:Crystal_GND24_Small
- C24: now not fitted; now left out of the parts list
- C5, C6: value 4.3p -> 0.1u; footprint Capacitor_SMD:C_0603_1608Metric -> Capacitor_SMD:C_0603_1608Metric_Pad1.08x0.95mm_HandSolder; PN GRM1885C1H4R3BA01D -> CL10B104KO8NNNC
- R32: value 4k7 -> 12.1k; PN ERJ-3EKF4701V -> RC0603FR-0712K4L; now fitted
- R33: value 4k7 -> 10k; footprint Resistor_SMD:R_0603_1608Metric_Pad0.98x0.95mm_HandSolder -> Resistor_SMD:R_0603_1608Metric; PN ERJ-3EKF4701V -> (none); now fitted
Connections:
- net SPI2_MISO is gone; now on net SDI_ENC: U5.3 (MISO)
- net SPI2_MOSI is gone; now on net SDO_ENC: U5.4 (MOSI)
- net SPI2_NSS is gone; now on net NSCS_ENC: U5.1 (CSn)
- net SPI2_SCK is gone; now on net SCLK_ENC: U5.2 (CLK)
- net +3V3: now also J6.P2, J6.P5, R33.1, U6.1 (VBAT), U6.13 (VDDA), U6.19 (VDD), U6.32 (VDD), U6.48 (VDD), U6.64 (VDD), U8.19 (NFREEZE), U8.26 (VCC), U8.37 (VCC), U8.5 (VCC), U9.1 (VDD2A), U9.19 (VDD1A), U9.9 (VDDIO), C46.1, C52.2, C53.2, C54.2, C55.2, C56.2, C57.1, C58.1, C59.1, C60.2, R38.1, R42.1, R43.1, R44.1; no longer R32.2, R33.2
- net CSN: now also U6.58 (PB6), U8.2 (NSCSIN); no longer U4.13 (CSN_CFG3)
- net DRV_ENN: now also U6.27 (PB1)
- net GND: now also C6.1, J6.P8, J6.SH1 (SHIELD), J6.SH2 (SHIELD__1), R32.1, U6.12 (VSSA), U6.18 (VSS), U6.31 (VSS), U6.47 (VSS), U6.60 (BOOT0), U6.63 (VSS), U8.15 (GND), U8.25 (GND), U8.34 (TEST_MODE), U8.36 (GND), U8.6 (GND), U9.25 (EPAD), C44.1, C45.2, C46.2, C47.1, C48.1, C49.2, C50.2, C51.2, C52.1, C53.1, C54.1, C55.1, C56.1, C57.2, C58.2, C59.2, C60.1, C61.1, C62.1, R36.2, R37.2, Y2.2, Y2.4; no longer C6.2
- net NRST: now also U6.7 (NRST)
- net ON_INDICATOR: now also U6.11 (PC3)
- net Out_1: now also C5.1, U8.12 (STOPL)
- net Out_2: now also C6.2, U8.14 (STOPR)
- net RXD: now also U6.44 (PA11)
- net SCK: now also U6.55 (PB3(JTDO), U8.3 (SCKIN); no longer U4.14 (SCK_CFG2)
- net SENSOR_INDICATOR: now also U6.10 (PC2)
- net SPI_MISO: now also U6.56 (PB4(NJTRST)), U8.7 (SDOIN); no longer U4.16 (SDO_CFG0)
- net SPI_MOSI: now also U6.57 (PB5), U8.4 (SDIIN); no longer U4.15 (SDI_CFG1)
- net SWCLK: now also U6.49 (PA14(JTCK)
- net SWDIO: now also U6.46 (PA13(JTMS)
- net TXD: now also U6.45 (PA12)
- net UART_RX: now also U6.43 (PA10)
- net UART_TX: now also U6.42 (PA9)
- net TXP: now reaches J6.P1
- net TXP: now also U9.21 (TXP), R42.2
- net at J6.P10: now also R36.1
- net LED2: now reaches J6.P11
- net LED2: now also U9.2 (LED2/NINT/NPME/*NINTSEL)
- net at J6.P12: now also R37.1
- net TXN: now reaches J6.P3
- net TXN: now also U9.20 (TXN), R38.2
- net RXP: now reaches J6.P4
- net RXP: now also U9.23 (RXP), R44.2
- net RXN: now reaches J6.P6
- net RXN: now also U9.22 (RXN), R43.2
- net LED1: now reaches J6.P9
- net LED1: now also U9.3 (LED1/NINT/NPME/*REGOFF)
- net at U9.11 (CRS_DV/*MODE2): now also R47.1
- net ETH_MDIO: now reaches U9.12 (MDIO)
- net ETH_MDIO: now also U6.16 (PA2)
- net ETH_MDC: now reaches U9.13 (MDC)
- net ETH_MDC: now also U6.9 (PC1)
- net ETH_REF_CLK: now reaches U9.14 (NINT/REFCLKO)
- net ETH_REF_CLK: now also U6.15 (PA1)
- net LAN_NRST: now reaches U9.15 (NRST)
- net LAN_NRST: now also R33.2, U6.17 (PA3), C49.1
- net ETH_TX_EN: now reaches U9.16 (TXEN)
- net ETH_TX_EN: now also U6.21 (PA5)
- net ETH_TXD0: now reaches U9.17 (TXD0)
- net ETH_TXD0: now also U6.33 (PB12)
- net ETH_TXD1: now reaches U9.18 (TXD1)
- net ETH_TXD1: now also U6.36 (PB15)
- net at U9.24 (RBIAS): now also R32.2
- net CLKIN: now reaches U9.5 (XTAL1/CLKIN)
- net CLKIN: now also U6.40 (PC9)
- net VDDCR: now reaches U9.6 (VDDCR)
- net VDDCR: now also C50.1, C51.1
- net at U9.7 (RXD1/*MODE1): now also R45.1
- net at U9.8 (RXD0/*MODE0): now also R46.1
- net ETH_CRS_DV: now reaches U6.23 (PA7)
- net ETH_CRS_DV: now also R47.2
- net ETH_RXD0: now reaches U6.24 (PC4)
- net ETH_RXD0: now also R46.2
- net ETH_RXD1: now reaches U6.25 (PC5)
- net ETH_RXD1: now also R45.2
- net TARGET_REACHED: now reaches U6.26 (PB0)
- net TARGET_REACHED: now also U8.31 (TARGET_REACHED)
- net INTR: now reaches U6.28 (PB2)
- net INTR: now also U8.33 (INTR)
- net at U6.30 (VCAP): now also U6.62 (VCAP), C44.2, C45.1
- net CLK_EXT: now reaches U6.41 (PA8)
- net CLK_EXT: now also U8.38 (CLK_EXT)
- net at U6.5 (PH0): now also C47.2, Y2.3
- net at U6.6 (PH1): now also C48.2, Y2.1
- net NSCS_ENC: now reaches U8.1 (ANEG_NSCLK)
- net SDI_ENC: now reaches U8.10 (B_SDI)
- net SDO_ENC: now reaches U8.11 (BNEG_NSDI)
- net at U8.16 (VDD1V8): now also C62.2
- net SPI_MOSI_DRV: now reaches U8.27 (SDODRV_SCLK)
- net SPI_MOSI_DRV: now also U4.15 (SDI_CFG1)
- net SPI_MISO_DRV: now reaches U8.28 (SDIDRV_NSCLK)
- net SPI_MISO_DRV: now also U4.16 (SDO_CFG0)
- net SCK_DRV: now reaches U8.29 (SCKDRV_NSDO)
- net SCK_DRV: now also U4.14 (SCK_CFG2)
- net CSN_DRV: now reaches U8.30 (NSCSDRV_SDO)
- net CSN_DRV: now also U4.13 (CSN_CFG3)
- net at U8.35 (VDD1V8): now also C61.2
- net SCLK_ENC: now reaches U8.40 (A_SCLK)
- no-connect marks 31 -> 32
Other:
- note added: "Search: LAN8742 RMII PHY Customer Evaluation Board Schematic"
- note added: "exposed pad must be connected to the ground plane with a via array."
- note removed: "will be migrating to STM32H563RGT6"
- moved on the sheet: C10, C2, C36, C37, C39, C7, C8, J6, U5, U6, U8, U9
Changed lines of the file:
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@@
 	(generator "eeschema")
 	(generator_version "8.0")
-	(paper "A2")
+	(paper "A1")

Commit message: internal stm32 usb added
Parts:
- removed C40, C42, C43: 0.1u, Capacitor_SMD:C_0603_1608Metric_Pad1.08x0.95mm_HandSolder, symbol Device:C
- removed C41: 4.7u, Capacitor_SMD:C_0603_1608Metric_Pad1.08x0.95mm_HandSolder, symbol Device:C
- removed R39: 1k, Resistor_SMD:R_0603_1608Metric, symbol Device:R
- removed R40: 22.1k, Resistor_SMD:R_0603_1608Metric, symbol Device:R
- removed R41: 47.5, Resistor_SMD:R_0603_1608Metric, symbol Device:R
- removed U7: CP2102N-Axx-xQFN24, Package_DFN_QFN:QFN-24-1EP_4x4mm_P0.5mm_EP2.6x2.6mm, symbol Interface_USB:CP2102N-Axx-xQFN24
- added D9: D_Schottky, Diode_SMD:D_SOD-128, symbol Device:D_Schottky
Connections:
- net D+: now also U6.45 (PA12)
- net D-: now also U6.44 (PA11)
- net RXD: now also U6.61 (PB8); no longer U6.44 (PA11)
- net TXD: now also U6.59 (PB7); no longer U6.45 (PA12)
- net Vm: now also D9.1 (K)
- net at D8.4 (K), J5.1 (VBUS): now also D9.2 (A)
- net UART_RX: no longer names the net of U6.43 (PA10)
- net UART_TX: no longer names the net of U6.42 (PA9)
Other:
- moved on the sheet: C10, C2, C34, C35, C37, C46, C7, C8, D8, J5, R28, R29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

Commit message: ver 2 design not finished
Parts:
- removed R45, R46, R47: 100, Resistor_SMD:R_0603_1608Metric, symbol Device:R_Small
- added C40: 47u, Capacitor_SMD:C_1206_3216Metric, symbol Device:C_Small
- added J8: Conn_01x05, Connector_PinHeader_2.54mm:PinHeader_1x05_P2.54mm_Vertical, symbol Connector_Generic:Conn_01x05
- C23, C49, R33: now not fitted
- J7: value Conn_01x05 -> P13-1123; footprint Connector_PinHeader_2.54mm:PinHeader_1x05_P2.54mm_Vertical -> pogo_pin_SWD:pogo_pin_SWD; PN (none) -> P13-1123; now fitted; now in the parts list
Connections:
- net ETH_CRS_DV: now also U9.11 (CRS_DV/*MODE2)
- net ETH_RXD0: now also U9.8 (RXD0/*MODE0)
- net ETH_RXD1: now also U9.7 (RXD1/*MODE1)
- net GND: now also C40.2
- net LAN_NRST: no longer U6.17 (PA3), U9.15 (NRST)
- net RXN: now also J6.P4; no longer J6.P6
- net RXP: now also J6.P6; no longer J6.P4
- net Vm: now also C40.1
- no-connect marks 32 -> 34
Other:
- note removed: "incremental ABI direct connection to TMC4361A-LA-T"
- moved on the sheet: C52, C53, C54, C56, R38, R42, R43, R44

Commit message: not finished
Parts:
- removed J8: Conn_01x05, Connector_PinHeader_2.54mm:PinHeader_1x05_P2.54mm_Vertical, symbol Connector_Generic:Conn_01x05
- added C41: 0.1u, Capacitor_SMD:C_0603_1608Metric_Pad1.08x0.95mm_HandSolder, symbol Device:C
- added J10, J11, J8, J9: Conn_02x06_Odd_Even, Connector_PinHeader_2.54mm:PinHeader_2x06_P2.54mm_Vertical, symbol Connector_Generic:Conn_02x06_Odd_Even
- added R39, R40, R41: 22, Resistor_SMD:R_0402_1005Metric, symbol Device:R_Small
- C10, C44, C45, C46, C50, C51, C57, C58, C59, C7: footprint Capacitor_SMD:C_0603_1608Metric_Pad1.08x0.95mm_HandSolder -> Capacitor_SMD:C_0402_1005Metric
- R32: footprint Resistor_SMD:R_0603_1608Metric_Pad0.98x0.95mm_HandSolder -> Resistor_SMD:R_0402_1005Metric
Connections:
- net +3V3: now also C41.2
- net CLK_EXT: now also R39.1; no longer U6.41 (PA8)
- net D+: now also R41.1; no longer U6.45 (PA12)
- net D-: now also R40.2; no longer U6.44 (PA11)
- net GND: now also C41.1
- net RXD: now also J8.2 (Pin_2); no longer U6.61 (PB8)
- net TXD: now also J8.4 (Pin_4); no longer U6.59 (PB7)
- new net: R39.2, U6.41 (PA8)
- new net: R40.1, U6.44 (PA11)
- new net: R41.2, U6.45 (PA12)
- new net RXD1: J10.2 (Pin_2), U6.61 (PB8)
- new net TXD1: J10.4 (Pin_4), U6.59 (PB7)
Other:
- note added: "CON ON ETH SHIELD"
- note added: "CONN ON DRIVER BOARD"
- moved on the sheet: C10, C2, C37, C46, C7, C8, D8, D9, J5

Commit message: not finish
Parts:
- added C42, C43: 22uF, Capacitor_SMD:C_0805_2012Metric_Pad1.18x1.45mm_HandSolder, symbol Device:C_Small
- added D10: D_Schottky, Diode_SMD:D_MicroSMP_AK, symbol Device:D_Schottky
- C4: footprint Capacitor_SMD:C_0603_1608Metric_Pad1.08x0.95mm_HandSolder -> Capacitor_SMD:C_0402_1005Metric
- D9: footprint Diode_SMD:D_SOD-128 -> Diode_SMD:D_MicroSMP_AK; PN (none) -> MSS1P6-M3/89A
Connections:
- net +3V3: now also J10.12 (Pin_12), J11.11 (Pin_11), J8.12 (Pin_12), J9.11 (Pin_11), C42.1, C43.1
- net CLK_EXT: now also J9.7 (Pin_7); no longer R39.1
- net CSN: now also J9.1 (Pin_1); no longer U6.58 (PB6)
- net DRV_ENN: now also U6.2 (PC13); no longer U6.27 (PB1)
- net GND: now also J10.1 (Pin_1), J10.10 (Pin_10), J10.3 (Pin_3), J10.6 (Pin_6), J10.9 (Pin_9), J11.10 (Pin_10), J11.9 (Pin_9), J8.1 (Pin_1), J8.10 (Pin_10), J8.3 (Pin_3), J8.6 (Pin_6), J8.9 (Pin_9), J9.10 (Pin_10), J9.9 (Pin_9), C42.2, C43.2
- net INTR: now also U6.4 (PC15); no longer U6.28 (PB2)
- net SCK: now also J9.5 (Pin_5); no longer U6.55 (PB3(JTDO)
- net SENSOR_INDICATOR: now also U6.8 (PC0); no longer U6.10 (PC2)
- net SPI_MISO: now also J9.4 (Pin_4); no longer U6.56 (PB4(NJTRST))
- net SPI_MOSI: now also J9.2 (Pin_2); no longer U6.57 (PB5)
- net TARGET_REACHED: now also U6.3 (PC14); no longer U6.26 (PB0)
- net Vm: now also D10.2 (A); no longer C1.1, D9.1 (K), R1.2, U1.3 (VIN), U1.4 (EN)
- net CSN_1: now reaches J11.1 (Pin_1)
- net CSN_1: now also U6.58 (PB6)
- net SPI_MOSI_1: now reaches J11.2 (Pin_2)
- net SPI_MOSI_1: now also U6.57 (PB5)
- net SPI_MISO_1: now reaches J11.4 (Pin_4)
- net SPI_MISO_1: now also U6.56 (PB4(NJTRST))
- net SCK_1: now reaches J11.5 (Pin_5)
- net SCK_1: now also U6.55 (PB3(JTDO)
- net CLK_EXT_1: now reaches J11.7 (Pin_7)
- net CLK_EXT_1: now also R39.1
- net PGOOD: now reaches J10.11 (Pin_11)
- net PGOOD: now also C1.1, D9.1 (K), J8.11 (Pin_11), R1.2, U1.3 (VIN), U1.4 (EN), D10.1 (K)
Other:
- moved on the sheet: C1, C3, D1, J10, J11, J8, J9, R1, U1

Commit message: not ready
Parts:
- removed C4: 0.1u, Capacitor_SMD:C_0402_1005Metric, symbol Device:C
- removed J7: P13-1123, pogo_pin_SWD:pogo_pin_SWD, symbol Connector_Generic:Conn_01x05
- added J12: Conn_01x02_Pin, Connector_PinHeader_1.27mm:PinHeader_1x02_P1.27mm_Vertical, symbol Connector:Conn_01x02_Pin
- added J13: Conn_01x03_Pin, Connector_PinHeader_1.27mm:PinHeader_1x03_P1.27mm_Vertical, symbol Connector:Conn_01x03_Pin
- added TH1: Thermistor_NTC, Resistor_SMD:R_0603_1608Metric, symbol Device:Thermistor_NTC
- C5, C6: footprint Capacitor_SMD:C_0603_1608Metric_Pad1.08x0.95mm_HandSolder -> Capacitor_SMD:C_0402_1005Metric
- D2: value LED_AMBER -> LED_ORANGE; footprint Diode_SMD:D_0603_1608Metric_Pad1.05x0.95mm_HandSolder -> LED_SMD:LED_0402_1005Metric; PN ASMT-RA45-AP932 -> SML-P11DTT86R
- D3: footprint Diode_SMD:D_0603_1608Metric_Pad1.05x0.95mm_HandSolder -> Diode_SMD:D_0402_1005Metric; PN SML-E12M8WT86 -> SML-P13PTT86R
- R2, R3: footprint Resistor_SMD:R_0603_1608Metric_Pad0.98x0.95mm_HandSolder -> Resistor_SMD:R_0402_1005Metric
Connections:
- net +3V3: now also J10.8 (Pin_8), J8.8 (Pin_8), J12.1 (Pin_1); no longer J10.12 (Pin_12), J8.12 (Pin_12)
- net CLK_EXT: now also U4.12 (CLK)
- net DRV_ENN: now also J8.5 (Pin_5); no longer U6.2 (PC13)
- net GND: now also J10.12 (Pin_12), J11.3 (Pin_3), J8.12 (Pin_12), J9.3 (Pin_3), J12.2 (Pin_2); no longer U4.12 (CLK)
- net INTR: now also J8.7 (Pin_7); no longer U6.4 (PC15)
- net NRST: now also J13.1 (Pin_1)
- net PGOOD: no longer D9.1 (K), J10.11 (Pin_11)
- net SWCLK: now also J13.2 (Pin_2)
- net SWDIO: now also J13.3 (Pin_3)
- net DRV_ENN_1: now reaches J10.5 (Pin_5)
- net DRV_ENN_1: now also U6.2 (PC13)
- net INTR_1: now reaches J10.7 (Pin_7)
- net INTR_1: now also U6.4 (PC15)
- net TARGET_REACHED: no longer names the net of U6.3 (PC14)
- net TARGET_REACHED: no longer U8.31 (TARGET_REACHED)
- new net PGOOD1: D9.1 (K), J10.11 (Pin_11)
