File: TMCM_1260_alternative_ver_2/TMCM_1260_alternative_ver_2.kicad_sch (KiCad schematic)
At the start: 140 parts, among them J1 Motor, J10 Conn_02x06_Odd_Even, J11 Conn_02x06_Odd_Even, J12 Conn_01x02_Pin, J13 Conn_01x03_Pin, J2 CAN, J3 I/O, J4 Power, J5 USB_B_Micro, J6 JXD2-0Z10NL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

Commit message: upload
Parts:
- removed R26: 2R2, Resistor_SMD:R_0603_1608Metric, symbol Device:R_Small
- C5, C6: footprint Capacitor_SMD:C_0402_1005Metric -> Capacitor_SMD:C_0603_1608Metric
Connections:
- net STOP_L/STEP is gone; now on net GND: J3.5 (Pin_5)
- net VCC_IO is gone; now on net +3V3: C33.1, R30.2, R31.1, U4.20 (VCC_IO), U4.22 (SPI_MODE)
- net +3V3: now also J11.8 (Pin_8), J9.8 (Pin_8), R34.2, R35.2
- net 5VOUT: no longer R34.2, R35.2
- net GND: now also J11.6 (Pin_6), J9.6 (Pin_6)
- net Out_1: now also J3.3 (Pin_3); no longer J3.2 (Pin_2)
- net Out_2: now also J3.2 (Pin_2); no longer J3.3 (Pin_3)
Other:
- moved on the sheet: C2, D2, D3, J12, J13, J8, J9, R2, R3

Commit message: finished not checked
Parts:
- removed C10, C57, C58, C59, C7: 0.1u, Capacitor_SMD:C_0402_1005Metric, symbol Device:C
- removed C37, C49, C8: 0.1u, Capacitor_SMD:C_0603_1608Metric_Pad1.08x0.95mm_HandSolder, symbol Device:C
- removed C42, C43: 22uF, Capacitor_SMD:C_0805_2012Metric_Pad1.18x1.45mm_HandSolder, symbol Device:C_Small
- removed C44, C45: 2.2u, Capacitor_SMD:C_0402_1005Metric, symbol Device:C
- removed C46: 4.7u, Capacitor_SMD:C_0402_1005Metric, symbol Device:C
- removed C47, C48: 15p, Capacitor_SMD:C_0603_1608Metric, symbol Device:C
- removed C50: 470p, Capacitor_SMD:C_0402_1005Metric, symbol Device:C
- removed C51: 1u, Capacitor_SMD:C_0402_1005Metric, symbol Device:C
- removed C52, C53, C54, C56: 10pF, Capacitor_SMD:C_0603_1608Metric_Pad1.08x0.95mm_HandSolder, symbol Device:C
- removed C55: 0.022uF, Capacitor_SMD:C_0603_1608Metric_Pad1.08x0.95mm_HandSolder, symbol Device:C
- removed D2: LED_ORANGE, LED_SMD:LED_0402_1005Metric, symbol Device:LED
- removed D3: LED_GREEN, Diode_SMD:D_0402_1005Metric, symbol Device:LED
- removed D8: SP0503BAHT, Package_TO_SOT_SMD:SOT-143, symbol Power_Protection:SP0503BAHT
- removed D9: D_Schottky, Diode_SMD:D_MicroSMP_AK, symbol Device:D_Schottky
- removed J10, J11: Conn_02x06_Odd_Even, Connector_PinHeader_2.54mm:PinHeader_2x06_P2.54mm_Vertical, symbol Connector_Generic:Conn_02x06_Odd_Even
- removed J12: Conn_01x02_Pin, Connector_PinHeader_1.27mm:PinHeader_1x02_P1.27mm_Vertical, symbol Connector:Conn_01x02_Pin
- removed J13: Conn_01x03_Pin, Connector_PinHeader_1.27mm:PinHeader_1x03_P1.27mm_Vertical, symbol Connector:Conn_01x03_Pin
- removed J5: USB_B_Micro, Connector_USB:USB_Micro-B_Molex-105133-0031, symbol Connector:USB_B_Micro
- removed J6: JXD2-0Z10NL, JXD2_0Z10NL:JXD2_0Z10NL, symbol JXD2-0Z10NL:JXD2-0Z10NL
- removed R3: 270, Resistor_SMD:R_0402_1005Metric, symbol Device:R_Small
- removed R32: 12.1k, Resistor_SMD:R_0402_1005Metric, symbol Device:R_Small
- removed R33: 10k, Resistor_SMD:R_0603_1608Metric, symbol Device:R_Small
- removed R36, R37: 330, Resistor_SMD:R_0603_1608Metric, symbol Device:R_Small
- removed R38, R42, R43, R44: 49.9, Resistor_SMD:R_0603_1608Metric, symbol Device:R_Small
- removed R39, R40, R41: 22, Resistor_SMD:R_0402_1005Metric, symbol Device:R_Small
- removed U6: STM32H563RGTx, Package_QFP:LQFP-64_10x10mm_P0.5mm, symbol MCU_ST_STM32H5:STM32H563RGTx
- removed U9: LAN8742A-CZ-TR, LAN8742A_CZ_TR:LAN8742A_CZ_TR, symbol LAN8742A_CZ_TR:LAN8742A-CZ-TR
- removed Y2: 25Mhz, Crystal:Crystal_SMD_2016-4Pin_2.0x1.6mm, symbol Device:Crystal_GND24_Small
- R2: value 270 -> 10k; footprint Resistor_SMD:R_0402_1005Metric -> Resistor_SMD:R_0603_1608Metric_Pad0.98x0.95mm_HandSolder; PN RMCF0603FT270R -> ERJ-3EKF4701V
Connections:
- net +3V3: now also TH1.2; no longer R2.2
- net GND: now also R2.1
- net monitoring: now reaches J9.12 (Pin_12)
- net monitoring: now also R2.2, TH1.1
- no-connect marks 34 -> 28
Other:
- note removed: "CON ON ETH SHIELD"
- note removed: "EXTERNAL shield that connects via pins on driver board and fixed with one screw"
- note removed: "Search: LAN8742 RMII PHY Customer Evaluation Board Schematic"
- note removed: "exposed pad must be connected to the ground plane with a via array."
- moved on the sheet: C1, C11, C3, C38, C5, C6, C9, D1, D10, R1, R34, R35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

Commit message: updated
Parts:
- added Q5, Q6, Q7: TLP185GR-TPL_SE, TLP185_GR_TPL_SE:TLP185_GR_TPL_SE, symbol TLP185_GR_TPL_SE:TLP185GR-TPL_SE
- added R3: 4k7, Resistor_SMD:R_0603_1608Metric_Pad0.98x0.95mm_HandSolder, symbol Device:R_Small
Connections:
- net IN2/ENC_B is gone; now on net Out_2: J3.4 (Pin_4)
- net +3V3: now also R3.2
- net 5VOUT: no longer J3.7 (Pin_7)
- net GND: no longer J3.6 (Pin_6)
- net Out_1: now also Q7.3
- net Out_2: now also Q6.3; no longer J3.2 (Pin_2)
- net Vm: now also J3.6 (Pin_6), J3.7 (Pin_7)
- net HOME_REF: now reaches U8.13 (HOME_REF)
- net HOME_REF: now also J3.2 (Pin_2), Q5.3, R3.1
- no-connect marks 28 -> 27
Other:
- moved on the sheet: C38, C5, C6, R34, R35

Commit message: finished
Parts:
- removed C6: 0.1u, Capacitor_SMD:C_0603_1608Metric, symbol Device:C
- added C4, C7: 0.1u, Capacitor_SMD:C_0402_1005Metric, symbol Device:C
- added R26, R32, R33: 24k, Resistor_SMD:R_0402_1005Metric, symbol Device:R_Small
- C5: footprint Capacitor_SMD:C_0603_1608Metric -> Capacitor_SMD:C_0402_1005Metric
- R3, R34, R35: footprint Resistor_SMD:R_0603_1608Metric_Pad0.98x0.95mm_HandSolder -> Resistor_SMD:R_0402_1005Metric
Connections:
- net GND: now also Q5.4, Q6.4, Q7.4, C4.2, C7.2
- net HOME_REF: now also Q5.6, C4.1; no longer J3.2 (Pin_2), Q5.3
- net Out_1: now also J3.4 (Pin_4); no longer C5.1, J3.3 (Pin_3), R35.1, U8.12 (STOPL)
- net Out_2: now also J3.3 (Pin_3); no longer J3.4 (Pin_4), R34.1, U8.14 (STOPR)
- net Vm: now also R26.2, R32.2, R33.2
- net at Q6.1: now also R32.1
- net STOPR: now reaches Q6.6
- net STOPR: now also C5.1, R34.1, U8.14 (STOPR)
- net at Q7.1: now also R33.1
- net STOPL: now reaches Q7.6
- net STOPL: now also R35.1, U8.12 (STOPL), C7.1
- net at Q5.1: now also R26.1
- new net home: J3.2 (Pin_2), Q5.3
Other:
- moved on the sheet: C38, Q5, Q6, Q7, R3

Commit message: absolute encoder SPI switched to ABI incremental
Parts:
- added C8: 0.1u, Capacitor_SMD:C_0603_1608Metric, symbol Device:C
- added R36, R37, R38: 4k7, Resistor_SMD:R_0402_1005Metric, symbol Device:R_Small
Connections:
- net +3V3: now also C8.1, R36.2
- net GND: now also U8.1 (ANEG_NSCLK), U8.11 (BNEG_NSDI), U8.22 (NNEG), C8.2, R37.2, R38.2
- net INCR_I: now reaches U5.14 (I/PWM)
- net INCR_I: now also U8.21 (N)
- net INCR_B: now reaches U5.6 (B)
- net INCR_B: now also U8.10 (B_SDI)
- net INCR_A: now reaches U5.7 (A)
- net INCR_A: now also U8.40 (A_SCLK)
- net NSCS_ENC: no longer names the net of U5.1 (CSn)
- net NSCS_ENC: now also R36.1; no longer U8.1 (ANEG_NSCLK)
- net SCLK_ENC: no longer names the net of U5.2 (CLK)
- net SCLK_ENC: now also R37.1; no longer U8.40 (A_SCLK)
- net SDI_ENC: no longer names the net of U5.3 (MISO)
- net SDI_ENC: no longer U8.10 (B_SDI)
- net SDO_ENC: no longer names the net of U5.4 (MOSI)
- net SDO_ENC: now also R38.1; no longer U8.11 (BNEG_NSDI)
- no-connect marks 27 -> 23
Other:
- moved on the sheet: C11, C9

Commit message: upload
Parts:
- C40: value 47u -> 22u
- R26, R32, R33: value 24k -> 2k4; PN ERJ-3EKF4701V -> ERJ-2GEJ242X
