File: TMCM_1260_alternative_ver_2/TMCM_1260_alternative_ver_2.kicad_pcb (KiCad board)
At the start: 4 copper layers, 60 x 60 mm, 97 parts, among them J1 Motor, J2 CAN, J3 I/O, J4 Power, J5 USB_B_Micro, J6 JXD2-0Z10NL, J7 Conn_01x05, Q1 NVMFD5C650NLT1G, Q2 NVMFD5C650NLT1G, Q3 NVMFD5C650NLT1G, Q4 NVMFD5C650NLT1G, U1 LMZM23600V3SILR, U2 STM32F091CCTx, U3 TCAN337, U4 TMC5160A-TA-T, U5 AS5047P-ATSM, U6 STM32H563RGTx, U7 CP2102N-Axx-xQFN24, U8 TMC4361A-LA-T, U9 LAN8742A-CZ-TR, Y1 Crystal_Small

Commit message: upload
Parts:
- moved J6 5.12 mm to (131.4, 129.8)
Connections:
- U2 pad 18: PB0 -> unconnected-(U2-PB0-Pad18)
- U2 pad 19: PB1 -> unconnected-(U2-PB1-Pad19)
- U2 pad 20: PB2 -> unconnected-(U2-PB2-Pad20)

Commit message: tmc4361 added ver_2
Parts:
- removed C24: 330u, Capacitor_THT:CP_Radial_D10.0mm_P5.00mm
- removed U2: STM32F091CCTx, Package_QFP:LQFP-48_7x7mm_P0.5mm
- added C44: 2.2u, Capacitor_SMD:C_0603_1608Metric_Pad1.08x0.95mm_HandSolder, F.Cu at (54.8, 110.2)
- added C45: 2.2u, Capacitor_SMD:C_0603_1608Metric_Pad1.08x0.95mm_HandSolder, F.Cu at (54.8, 112.7)
- added C46: 4.7u, Capacitor_SMD:C_0603_1608Metric_Pad1.08x0.95mm_HandSolder, F.Cu at (54.8, 115.2)
- added C47: 15p, Capacitor_SMD:C_0603_1608Metric, F.Cu at (54.7, 122.7)
- added C48: 15p, Capacitor_SMD:C_0603_1608Metric, F.Cu at (54.7, 125.2)
- added C49: 0.1u, Capacitor_SMD:C_0603_1608Metric_Pad1.08x0.95mm_HandSolder, F.Cu at (54.8, 117.7)
- added C50: 470p, Capacitor_SMD:C_0603_1608Metric_Pad1.08x0.95mm_HandSolder, F.Cu at (54.8, 120.2)
- added C51: 1u, Capacitor_SMD:C_0603_1608Metric_Pad1.08x0.95mm_HandSolder, F.Cu at (59.2, 110.2)
- added C52: 10pF, Capacitor_SMD:C_0603_1608Metric_Pad1.08x0.95mm_HandSolder, F.Cu at (59.2, 112.7)
- added C53: 10pF, Capacitor_SMD:C_0603_1608Metric_Pad1.08x0.95mm_HandSolder, F.Cu at (59.2, 115.2)
- added C54: 10pF, Capacitor_SMD:C_0603_1608Metric_Pad1.08x0.95mm_HandSolder, F.Cu at (59.2, 117.7)
- added C55: 0.022uF, Capacitor_SMD:C_0603_1608Metric_Pad1.08x0.95mm_HandSolder, F.Cu at (59.2, 120.2)
- added C56: 10pF, Capacitor_SMD:C_0603_1608Metric_Pad1.08x0.95mm_HandSolder, F.Cu at (63.5, 110.2)
- added C57: 0.1u, Capacitor_SMD:C_0603_1608Metric_Pad1.08x0.95mm_HandSolder, F.Cu at (63.5, 112.7)
- added C58: 0.1u, Capacitor_SMD:C_0603_1608Metric_Pad1.08x0.95mm_HandSolder, F.Cu at (63.5, 115.2)
- added C59: 0.1u, Capacitor_SMD:C_0603_1608Metric_Pad1.08x0.95mm_HandSolder, F.Cu at (63.5, 117.7)
- added R32: 12.1k, Resistor_SMD:R_0603_1608Metric_Pad0.98x0.95mm_HandSolder, F.Cu at (63.5, 120.2)
- added R33: 10k, Resistor_SMD:R_0603_1608Metric, F.Cu at (54.7, 127.7)
- added R36: 330, Resistor_SMD:R_0603_1608Metric, F.Cu at (54.7, 130.3)
- added R37: 330, Resistor_SMD:R_0603_1608Metric, F.Cu at (58.7, 122.7)
- added R38: 49.9, Resistor_SMD:R_0603_1608Metric, F.Cu at (58.7, 125.2)
- added R42: 49.9, Resistor_SMD:R_0603_1608Metric, F.Cu at (58.7, 127.7)
- added R43: 49.9, Resistor_SMD:R_0603_1608Metric, F.Cu at (58.7, 130.3)
- added R44: 49.9, Resistor_SMD:R_0603_1608Metric, F.Cu at (62.7, 122.7)
- added R45: 100, Resistor_SMD:R_0603_1608Metric, F.Cu at (62.7, 125.2)
- added R46: 100, Resistor_SMD:R_0603_1608Metric, F.Cu at (62.7, 127.7)
- added R47: 100, Resistor_SMD:R_0603_1608Metric, F.Cu at (62.7, 130.3)
- added Y2: 25Mhz, Crystal:Crystal_SMD_2016-4Pin_2.0x1.6mm, F.Cu at (66.6, 123.3)
- Y1: value Crystal_Small -> 8Mhz
- moved U8 39.1 mm to (97.6, 120.7)
- moved J7 38.4 mm to (148.3, 99.9)
- moved U6 33.4 mm to (114.8, 115.7), turned to 180 degrees
- moved C10 30.5 mm to (138.9, 104.3)
- moved C7 20.5 mm to (134.2, 105.6)
- moved C37 15.5 mm to (136.1, 115.4)
- moved U9 11.4 mm to (145.4, 132.7)
- moved C16 3.40 mm to (105.5, 113.8)
Connections:
- C5 pad 1: Net-(U2-PF0) -> Net-(U6-PH0)
- C6 pad 1: Net-(U2-PF1) -> Net-(U6-PH1)
- J6 pad P1: unconnected-(J6-PadP1) -> TXP
- J6 pad P10: unconnected-(J6-PadP10) -> Net-(J6-PadP10)
- J6 pad P11: unconnected-(J6-PadP11) -> LED2
- J6 pad P12: unconnected-(J6-PadP12) -> Net-(J6-PadP12)
- J6 pad P2: unconnected-(J6-PadP2) -> +3V3
- J6 pad P3: unconnected-(J6-PadP3) -> TXN
- J6 pad P4: unconnected-(J6-PadP4) -> RXP
- J6 pad P5: unconnected-(J6-PadP5) -> +3V3
- J6 pad P6: unconnected-(J6-PadP6) -> RXN
- J6 pad P8: unconnected-(J6-PadP8) -> GND
- J6 pad P9: unconnected-(J6-PadP9) -> LED1
- J6 pad SH1: unconnected-(J6-SHIELD-PadSH1) -> GND
- J6 pad SH2: unconnected-(J6-SHIELD__1-PadSH2) -> GND
- U6 pad 1: unconnected-(U6-VBAT-Pad1) -> +3V3
- U6 pad 10: unconnected-(U6-PC2-Pad10) -> SENSOR_INDICATOR
- U6 pad 11: unconnected-(U6-PC3-Pad11) -> ON_INDICATOR
- U6 pad 12: unconnected-(U6-VSSA-Pad12) -> GND
- U6 pad 13: unconnected-(U6-VDDA-Pad13) -> +3V3
- U6 pad 15: unconnected-(U6-PA1-Pad15) -> ETH_REF_CLK
- U6 pad 16: unconnected-(U6-PA2-Pad16) -> ETH_MDIO
- U6 pad 18: Net-(U6-VSS-Pad18) -> GND
- U6 pad 19: unconnected-(U6-VDD-Pad19) -> +3V3
- U6 pad 20: unconnected-(U6-PA4-Pad20) -> CSN
- U6 pad 21: unconnected-(U6-PA5-Pad21) -> ETH_TX_EN
- U6 pad 22: unconnected-(U6-PA6-Pad22) -> SPI_MISO
- U6 pad 23: unconnected-(U6-PA7-Pad23) -> ETH_CRS_DV
- U6 pad 24: unconnected-(U6-PC4-Pad24) -> ETH_RXD0
- U6 pad 25: unconnected-(U6-PC5-Pad25) -> ETH_RXD1
- U6 pad 30: unconnected-(U6-VCAP-Pad30) -> Net-(C44-Pad2)
- U6 pad 31: Net-(U6-VSS-Pad18) -> GND
- U6 pad 32: unconnected-(U6-VDD-Pad32) -> +3V3
- U6 pad 33: unconnected-(U6-PB12-Pad33) -> ETH_TXD0
- U6 pad 34: unconnected-(U6-PB13-Pad34) -> SPI2_SCK
- U6 pad 35: unconnected-(U6-PB14-Pad35) -> SPI2_MISO
- U6 pad 36: unconnected-(U6-PB15-Pad36) -> ETH_TXD1
- U6 pad 42: unconnected-(U6-PA9-Pad42) -> UART_TX
- U6 pad 43: unconnected-(U6-PA10-Pad43) -> UART_RX
- U6 pad 44: unconnected-(U6-PA11-Pad44) -> /RXD
- U6 pad 45: unconnected-(U6-PA12-Pad45) -> /TXD
- U6 pad 46: unconnected-(U6-PA13(JTMS-Pad46) -> /SWDIO
- U6 pad 47: Net-(U6-VSS-Pad18) -> GND
- U6 pad 48: unconnected-(U6-VDD-Pad48) -> +3V3
- U6 pad 49: unconnected-(U6-PA14(JTCK-Pad49) -> /SWCLK
- U6 pad 5: unconnected-(U6-PH0-Pad5) -> Net-(U6-PH0)
- U6 pad 57: unconnected-(U6-PB5-Pad57) -> Out_2
- U6 pad 58: unconnected-(U6-PB6-Pad58) -> Out_1
- U6 pad 6: unconnected-(U6-PH1-Pad6) -> Net-(U6-PH1)
- U6 pad 60: unconnected-(U6-BOOT0-Pad60) -> GND
- U6 pad 62: unconnected-(U6-VCAP-Pad62) -> Net-(C44-Pad2)
- U6 pad 63: Net-(U6-VSS-Pad18) -> GND
- U6 pad 64: unconnected-(U6-VDD-Pad64) -> +3V3
- U6 pad 7: unconnected-(U6-NRST-Pad7) -> /NRST
- U6 pad 9: unconnected-(U6-PC1-Pad9) -> ETH_MDC
- U9 pad 1: unconnected-(U9-VDD2A-Pad1) -> +3V3
- U9 pad 11: unconnected-(U9-CRS_DV/*MODE2-Pad11) -> Net-(U9-CRS_DV/*MODE2)
- U9 pad 12: unconnected-(U9-MDIO-Pad12) -> ETH_MDIO
- U9 pad 13: unconnected-(U9-MDC-Pad13) -> ETH_MDC
- U9 pad 14: unconnected-(U9-NINT/REFCLKO-Pad14) -> ETH_REF_CLK
- U9 pad 15: unconnected-(U9-NRST-Pad15) -> LAN_NRST
- U9 pad 16: unconnected-(U9-TXEN-Pad16) -> ETH_TX_EN
- U9 pad 17: unconnected-(U9-TXD0-Pad17) -> ETH_TXD0
- U9 pad 18: unconnected-(U9-TXD1-Pad18) -> ETH_TXD1
- U9 pad 19: unconnected-(U9-VDD1A-Pad19) -> +3V3
- U9 pad 2: unconnected-(U9-LED2/NINT/NPME/*NINTSEL-Pad2) -> LED2
- U9 pad 20: unconnected-(U9-TXN-Pad20) -> TXN
- U9 pad 21: unconnected-(U9-TXP-Pad21) -> TXP
- U9 pad 22: unconnected-(U9-RXN-Pad22) -> RXN
- U9 pad 23: unconnected-(U9-RXP-Pad23) -> RXP
- U9 pad 24: unconnected-(U9-RBIAS-Pad24) -> Net-(U9-RBIAS)
- U9 pad 25: unconnected-(U9-EPAD-Pad25) -> GND
- U9 pad 3: unconnected-(U9-LED1/NINT/NPME/*REGOFF-Pad3) -> LED1
- U9 pad 4: unconnected-(U9-XTAL2-Pad4) -> Net-(U9-XTAL2)
- U9 pad 5: unconnected-(U9-XTAL1/CLKIN-Pad5) -> Net-(U9-XTAL1/CLKIN)
- U9 pad 6: unconnected-(U9-VDDCR-Pad6) -> VDDCR
- U9 pad 7: unconnected-(U9-RXD1/*MODE1-Pad7) -> Net-(U9-RXD1/*MODE1)
- U9 pad 8: unconnected-(U9-RXD0/*MODE0-Pad8) -> Net-(U9-RXD0/*MODE0)
- U9 pad 9: unconnected-(U9-VDDIO-Pad9) -> +3V3
- Y1 pad 1: Net-(U2-PF0) -> Net-(U6-PH0)
- Y1 pad 2: Net-(U2-PF1) -> Net-(U6-PH1)
Routing:
- net +3V3: track 157.3 -> 119.3 mm, vias 6 -> 5
- net /NRST: track 24.7 -> 0.86 mm, vias 3 -> 0
- net 5VOUT: track 73.0 -> 52.9 mm
- net UART_TX: track 34.8 -> 18.2 mm, vias 1 -> 0
- net /TXD: track 29.3 -> 12.7 mm, vias 2 -> 1
- net SPI2_MOSI: track 28.9 -> 12.5 mm, vias 1 -> 0
- net SRBL: track 21.9 -> 7.85 mm
- net /SWDIO: track 13.5 -> 0.00 mm, vias 1 -> 0
- net Out_2: track 23.7 -> 10.3 mm
- net SCK: track 15.3 -> 2.00 mm
- net Out_1: track 24.8 -> 11.7 mm
- net SRBH: track 18.9 -> 5.99 mm
- net UART_RX: track 31.3 -> 20.3 mm, vias 1 -> 0
- net SPI2_NSS: track 27.0 -> 16.5 mm, vias 1 -> 0
- net /RXD: track 18.7 -> 9.39 mm, vias 2 -> 1
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