File: TMCM_1260_alternative_ver_2/TMCM_1260_alternative_ver_2.kicad_pcb (KiCad board)
At the start: 4 copper layers, 60 x 60 mm, 115 parts, among them J1 Motor, J2 CAN, J3 I/O, J4 Power, J5 USB_B_Micro, J6 JXD2-0Z10NL, J7 P13-1123, J8 Conn_01x05, Q1 NVMFD5C650NLT1G, Q2 NVMFD5C650NLT1G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

Commit message: not finished
Parts:
- removed Y1: 8Mhz, digikey-footprints:SMD-2_3.2x2.5mm
- added C41: 0.1u, Capacitor_SMD:C_0603_1608Metric_Pad1.08x0.95mm_HandSolder, F.Cu at (152.8, 88.9)
- added J10: Conn_02x06_Odd_Even, Connector_PinHeader_2.54mm:PinHeader_2x06_P2.54mm_Vertical, F.Cu at (89.8, 63.5)
- added J11: Conn_02x06_Odd_Even, Connector_PinHeader_2.54mm:PinHeader_2x06_P2.54mm_Vertical, F.Cu at (82.9, 98.5)
- added J9: Conn_02x06_Odd_Even, Connector_PinHeader_2.54mm:PinHeader_2x06_P2.54mm_Vertical, F.Cu at (140.1, 99.3)
- added R39: 22, Resistor_SMD:R_0402_1005Metric, F.Cu at (68.3, 110.5)
- added R40: 22, Resistor_SMD:R_0402_1005Metric, F.Cu at (71.6, 109.9)
- added R41: 22, Resistor_SMD:R_0402_1005Metric, F.Cu at (74.8, 109.7)
- C10, C44, C46, C50, C51, C57, C58, C59, C7: footprint Capacitor_SMD:C_0603_1608Metric_Pad1.08x0.95mm_HandSolder -> Capacitor_SMD:C_0402_1005Metric
- C2, C37, C52, C53, C54, C56, C60, R38, R42, R43, R44: moved to B.Cu
- C45: footprint Capacitor_SMD:C_0603_1608Metric_Pad1.08x0.95mm_HandSolder -> Capacitor_SMD:C_0402_1005Metric; moved to B.Cu
- C5, C6: footprint Capacitor_SMD:C_0603_1608Metric -> Capacitor_SMD:C_0603_1608Metric_Pad1.08x0.95mm_HandSolder; moved to F.Cu
- J8: value Conn_01x05 -> Conn_02x06_Odd_Even; footprint Connector_PinHeader_2.54mm:PinHeader_1x05_P2.54mm_Vertical -> Connector_PinHeader_2.54mm:PinHeader_2x06_P2.54mm_Vertical
- R32: footprint Resistor_SMD:R_0603_1608Metric_Pad0.98x0.95mm_HandSolder -> Resistor_SMD:R_0402_1005Metric
- moved C53 99.5 mm to (56.3, 82.8), turned to -90 degrees
- moved R44 98.7 mm to (54.3, 91.2), turned to 90 degrees
- moved C52 98.4 mm to (51.1, 90.6)
- moved C54 96.6 mm to (61.0, 83.8)
- moved R38 96.1 mm to (58.1, 83.0), turned to -90 degrees
- moved C56 96.0 mm to (59.3, 92.1), turned to 180 degrees
- moved R43 95.2 mm to (56.8, 91.1), turned to 90 degrees
- moved R42 91.9 mm to (63.2, 85.8), turned to 180 degrees
- moved D9 82.4 mm to (63.1, 112.0), turned to 180 degrees
- moved C45 79.0 mm to (86.2, 81.1), turned to 0 degrees
- moved C44 75.3 mm to (78.1, 87.6)
- moved C51 67.8 mm to (73.6, 85.5)
- moved C58 67.7 mm to (69.2, 77.1), turned to 90 degrees
- moved C46 67.7 mm to (89.4, 75.4), turned to 90 degrees
- moved C50 67.4 mm to (73.6, 84.6)
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Connections:
- J8 pad 2: unconnected-(J8-Pin_2-Pad2) -> /RXD
- J8 pad 4: unconnected-(J8-Pin_4-Pad4) -> /TXD
- U6 pad 41: CLK_EXT -> Net-(U6-PA8)
- U6 pad 44: D- -> Net-(U6-PA11)
- U6 pad 45: D+ -> Net-(U6-PA12)
- U6 pad 59: /TXD -> /TXD1
- U6 pad 61: /RXD -> /RXD1
Routing:
- net +3V3: track 106.3 -> 179.2 mm, vias 5 -> 10
- net (no net): track 38.4 -> 0.00 mm, vias 11 -> 5
- net SDO_ENC: track 9.08 -> 44.2 mm, vias 0 -> 1
- net SDI_ENC: track 10.7 -> 43.1 mm, vias 0 -> 1
- net NSCS_ENC: track 12.9 -> 39.9 mm, vias 0 -> 1
- net Net-(C44-Pad2): track 0.00 -> 25.5 mm, vias 0 -> 2
- net SCLK_ENC: track 11.8 -> 35.8 mm, vias 0 -> 1
- net GND: track 43.1 -> 63.2 mm, vias 93 -> 155
- net SRBL: track 7.85 -> 22.7 mm
- net SRBH: track 5.99 -> 20.3 mm
- net DRV_ENN: track 25.2 -> 11.1 mm
- net SCK_DRV: track 2.00 -> 15.2 mm
- net Net-(D9-A): track 9.96 -> 0.00 mm
- net /RXD: track 9.39 -> 18.3 mm, vias 1 -> 0
- net D-: track 8.64 -> 0.00 mm
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Other:
- board size 60 x 60 mm -> 112.4 x 60 mm

Commit message: not finish
Parts:
- added C42: 22uF, Capacitor_SMD:C_0805_2012Metric_Pad1.18x1.45mm_HandSolder, F.Cu at (65.3, 94.6)
- added C43: 22uF, Capacitor_SMD:C_0805_2012Metric_Pad1.18x1.45mm_HandSolder, F.Cu at (78.3, 68.9)
- added D10: D_Schottky, Diode_SMD:D_MicroSMP_AK, B.Cu at (138.1, 55.8)
- C4: footprint Capacitor_SMD:C_0603_1608Metric_Pad1.08x0.95mm_HandSolder -> Capacitor_SMD:C_0402_1005Metric; moved to B.Cu
- D8: moved to F.Cu
- D9: footprint Diode_SMD:D_SOD-128 -> Diode_SMD:D_MicroSMP_AK; moved to B.Cu
- moved C4 53.7 mm to (88.8, 89.9)
- moved R39 26.1 mm to (84.2, 89.8), turned to 90 degrees
- moved D9 25.5 mm to (77.9, 91.2)
- moved R40 24.5 mm to (85.4, 89.7), turned to -90 degrees
- moved R41 23.1 mm to (86.4, 89.7), turned to 90 degrees
- moved D8 10.1 mm to (69.8, 94.4), turned to 180 degrees
- moved J7 7.10 mm to (90.2, 91.2), turned to 180 degrees
- moved J11 6.00 mm to (76.9, 98.5)
- moved J9 6.00 mm to (134.1, 99.3)
- moved C10 2.72 mm to (76.5, 85.3), turned to 90 degrees
- moved J5 2.38 mm to (71.6, 90.3), turned to 180 degrees
- moved C38 1.61 mm to (102.8, 104.1)
- moved C1 0.39 mm to (138.9, 54.3)
Connections:
- C1 pad 1: 12-36V -> PGOOD
- D9 pad 1: 12-36V -> PGOOD
- J10 pad 1: unconnected-(J10-Pin_1-Pad1) -> GND
- J10 pad 10: unconnected-(J10-Pin_10-Pad10) -> GND
- J10 pad 11: unconnected-(J10-Pin_11-Pad11) -> PGOOD
- J10 pad 12: unconnected-(J10-Pin_12-Pad12) -> +3V3
- J10 pad 3: unconnected-(J10-Pin_3-Pad3) -> GND
- J10 pad 6: unconnected-(J10-Pin_6-Pad6) -> GND
- J10 pad 9: unconnected-(J10-Pin_9-Pad9) -> GND
- J11 pad 1: unconnected-(J11-Pin_1-Pad1) -> CSN_1
- J11 pad 10: unconnected-(J11-Pin_10-Pad10) -> GND
- J11 pad 11: unconnected-(J11-Pin_11-Pad11) -> +3V3
- J11 pad 2: unconnected-(J11-Pin_2-Pad2) -> SPI_MOSI_1
- J11 pad 4: unconnected-(J11-Pin_4-Pad4) -> SPI_MISO_1
- J11 pad 5: unconnected-(J11-Pin_5-Pad5) -> SCK_1
- J11 pad 7: unconnected-(J11-Pin_7-Pad7) -> CLK_EXT_1
- J11 pad 9: unconnected-(J11-Pin_9-Pad9) -> GND
- J8 pad 1: unconnected-(J8-Pin_1-Pad1) -> GND
- J8 pad 10: unconnected-(J8-Pin_10-Pad10) -> GND
- J8 pad 11: unconnected-(J8-Pin_11-Pad11) -> PGOOD
- J8 pad 12: unconnected-(J8-Pin_12-Pad12) -> +3V3
- J8 pad 3: unconnected-(J8-Pin_3-Pad3) -> GND
- J8 pad 6: unconnected-(J8-Pin_6-Pad6) -> GND
- J8 pad 9: unconnected-(J8-Pin_9-Pad9) -> GND
- J9 pad 1: unconnected-(J9-Pin_1-Pad1) -> CSN
- J9 pad 10: unconnected-(J9-Pin_10-Pad10) -> GND
- J9 pad 11: unconnected-(J9-Pin_11-Pad11) -> +3V3
- J9 pad 2: unconnected-(J9-Pin_2-Pad2) -> SPI_MOSI
- J9 pad 4: unconnected-(J9-Pin_4-Pad4) -> SPI_MISO
- J9 pad 5: unconnected-(J9-Pin_5-Pad5) -> SCK
- J9 pad 7: unconnected-(J9-Pin_7-Pad7) -> CLK_EXT
- J9 pad 9: unconnected-(J9-Pin_9-Pad9) -> GND
- R1 pad 2: 12-36V -> PGOOD
- R39 pad 1: CLK_EXT -> CLK_EXT_1
- U1 pad 3: 12-36V -> PGOOD
- U1 pad 4: 12-36V -> PGOOD
- U6 pad 10: SENSOR_INDICATOR -> unconnected-(U6-PC2-Pad10)
- U6 pad 2: unconnected-(U6-PC13-Pad2) -> DRV_ENN
- U6 pad 26: TARGET_REACHED -> unconnected-(U6-PB0-Pad26)
- U6 pad 27: DRV_ENN -> unconnected-(U6-PB1-Pad27)
- U6 pad 28: INTR -> unconnected-(U6-PB2-Pad28)
- U6 pad 3: unconnected-(U6-PC14-Pad3) -> TARGET_REACHED
- U6 pad 4: unconnected-(U6-PC15-Pad4) -> INTR
- U6 pad 55: SCK -> SCK_1
- U6 pad 56: SPI_MISO -> SPI_MISO_1
- U6 pad 57: SPI_MOSI -> SPI_MOSI_1
- U6 pad 58: CSN -> CSN_1
- U6 pad 8: unconnected-(U6-PC0-Pad8) -> SENSOR_INDICATOR
Routing:
- net +3V3: track 179.2 -> 289.6 mm, vias 10 -> 19
- net PGOOD: track 0.00 -> 61.7 mm, vias 0 -> 1
- net SPI_MISO_1: track 0.00 -> 36.4 mm
- net SPI_MOSI_1: track 0.00 -> 35.5 mm
- net SCK_1: track 0.00 -> 34.2 mm
- net CSN_1: track 0.00 -> 33.6 mm
- net CLK_EXT_1: track 0.00 -> 28.5 mm
- net D-: track 0.00 -> 27.3 mm
- net SPI_MISO: track 0.00 -> 26.2 mm
- net SCK: track 0.00 -> 25.0 mm
- net /TXD1: track 0.00 -> 21.5 mm
- net D+: track 0.00 -> 20.4 mm
- net SPI_MOSI: track 0.00 -> 20.0 mm
- net CLK_EXT: track 6.12 -> 25.8 mm
- net Net-(D9-A): track 0.00 -> 19.5 mm, vias 0 -> 2
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Other:
- outline, holes or cut-outs redrawn

Commit message: not finished
Parts:
- R2, R3: footprint Resistor_SMD:R_0603_1608Metric_Pad0.98x0.95mm_HandSolder -> Resistor_SMD:R_0402_1005Metric
- moved D2 93.0 mm to (69.7, 67.3)
- moved D3 93.0 mm to (69.7, 68.9)
- moved R2 92.7 mm to (66.7, 67.3)
- moved R3 92.6 mm to (66.8, 68.8)
- moved C47 0.94 mm to (87.7, 72.1), turned to -90 degrees
Routing:
- net TARGET_REACHED: track 0.00 -> 15.0 mm, vias 0 -> 1
- net DRV_ENN: track 11.1 -> 25.5 mm
- net INTR: track 0.00 -> 12.1 mm, vias 0 -> 1
- net SENSOR_INDICATOR: track 0.00 -> 7.90 mm, vias 0 -> 2
- net ON_INDICATOR: track 0.00 -> 7.22 mm, vias 0 -> 2
- net +3V3: track 289.6 -> 287.4 mm
- net PGOOD: track 61.7 -> 62.6 mm
- net ETH_REF_CLK: track 16.5 -> 16.0 mm
- net GND: vias 154 -> 156
- net (no net): vias 5 -> 2

Commit message: not ready
Parts:
- removed J7: P13-1123, pogo_pin_SWD:pogo_pin_SWD
- added J12: Conn_01x02_Pin, Connector_PinHeader_1.27mm:PinHeader_1x02_P1.27mm_Vertical, F.Cu at (86.8, 77.6)
- added J13: Conn_01x03_Pin, Connector_PinHeader_1.27mm:PinHeader_1x03_P1.27mm_Vertical, F.Cu at (86.8, 80.1)
- added TH1: Thermistor_NTC, Resistor_SMD:R_0603_1608Metric, F.Cu at (104.1, 58.7)
- C5, C6: footprint Capacitor_SMD:C_0603_1608Metric_Pad1.08x0.95mm_HandSolder -> Capacitor_SMD:C_0402_1005Metric
- D2: value LED_AMBER -> LED_ORANGE; footprint Diode_SMD:D_0603_1608Metric_Pad1.05x0.95mm_HandSolder -> LED_SMD:LED_0402_1005Metric
- D3: footprint Diode_SMD:D_0603_1608Metric_Pad1.05x0.95mm_HandSolder -> Diode_SMD:D_0402_1005Metric
- R2, R3: moved to B.Cu
- moved C5 63.5 mm to (102.6, 110.4)
- moved C6 63.4 mm to (102.6, 112.4)
- moved C4 11.9 mm to (78.5, 83.9), turned to -90 degrees
- moved R2 11.0 mm to (76.5, 72.3), turned to 90 degrees
- moved R3 9.27 mm to (75.4, 72.3), turned to -90 degrees
- moved D2 9.07 mm to (76.5, 73.3), turned to 90 degrees
- moved D3 7.18 mm to (75.4, 73.3), turned to 90 degrees
- moved C7 6.56 mm to (83.6, 89.9), turned to 0 degrees
- moved C44 5.87 mm to (72.7, 89.8)
- moved C45 5.87 mm to (80.7, 83.3)
- moved C59 5.87 mm to (65.9, 88.2)
- moved U9 5.87 mm to (66.2, 83.5)
- moved C42 5.87 mm to (59.9, 96.8)
- moved C53 5.87 mm to (50.9, 85.0)
- moved C56 5.87 mm to (53.8, 94.3)
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Connections:
- D9 pad 1: PGOOD -> PGOOD1
- J10 pad 11: PGOOD -> PGOOD1
- J10 pad 12: +3V3 -> GND
- J10 pad 5: unconnected-(J10-Pin_5-Pad5) -> DRV_ENN_1
- J10 pad 7: unconnected-(J10-Pin_7-Pad7) -> INTR_1
- J10 pad 8: unconnected-(J10-Pin_8-Pad8) -> +3V3
- J11 pad 3: unconnected-(J11-Pin_3-Pad3) -> GND
- J8 pad 12: +3V3 -> GND
- J8 pad 5: unconnected-(J8-Pin_5-Pad5) -> DRV_ENN
- J8 pad 7: unconnected-(J8-Pin_7-Pad7) -> INTR
- J8 pad 8: unconnected-(J8-Pin_8-Pad8) -> +3V3
- J9 pad 3: unconnected-(J9-Pin_3-Pad3) -> GND
- U4 pad 12: GND -> CLK_EXT
- U6 pad 2: DRV_ENN -> DRV_ENN_1
- U6 pad 3: TARGET_REACHED -> unconnected-(U6-PC14-Pad3)
- U6 pad 4: INTR -> INTR_1
- U8 pad 31: TARGET_REACHED -> unconnected-(U8-TARGET_REACHED-Pad31)
Routing:
- net PGOOD: track 62.6 -> 14.0 mm
- net PGOOD1: track 0.00 -> 48.6 mm
- net +3V3: track 287.4 -> 312.1 mm
- net INTR_1: track 0.00 -> 18.9 mm, vias 0 -> 1
- net DRV_ENN_1: track 0.00 -> 16.0 mm
- net TARGET_REACHED: track 15.0 -> 0.00 mm, vias 1 -> 0
- net DRV_ENN: track 25.5 -> 11.1 mm
- net INTR: track 12.1 -> 0.00 mm, vias 1 -> 0
- net CLK_EXT: track 25.8 -> 37.5 mm
- net /SWDIO: track 4.27 -> 13.0 mm, vias 0 -> 1
- net CSN_1: track 33.6 -> 29.3 mm
- net GND: track 66.0 -> 61.7 mm, vias 156 -> 167
- net /SWCLK: track 7.68 -> 11.6 mm, vias 0 -> 1
- net SPI_MOSI_1: track 35.5 -> 32.1 mm
- net SPI_MISO_1: track 36.4 -> 33.2 mm
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Other:
- board size 112.4 x 60 mm -> 117.8 x 60 mm
- board text added: "3V3"

Commit message: upload
Parts:
- removed R26: 2R2, Resistor_SMD:R_0603_1608Metric
- C38, R34, R35: moved to B.Cu
- C5, C6: footprint Capacitor_SMD:C_0402_1005Metric -> Capacitor_SMD:C_0603_1608Metric; moved to B.Cu
- moved C6 32.5 mm to (134.6, 107.0), turned to 180 degrees
- moved R34 31.7 mm to (134.5, 105.5)
- moved C5 27.3 mm to (129.7, 107.0), turned to 180 degrees
- moved R35 27.0 mm to (129.8, 105.5), turned to 0 degrees
- moved C38 17.3 mm to (119.6, 108.4), turned to 90 degrees
Connections:
- C10 pad 1: +3V3 -> VCC_IO
- C11 pad 1: +3V3 -> VCC_IO
- C2 pad 1: +3V3 -> VCC_IO
- C3 pad 1: +3V3 -> VCC_IO
- C36 pad 2: +3V3 -> VCC_IO
- C37 pad 1: +3V3 -> VCC_IO
- C39 pad 2: +3V3 -> VCC_IO
- C41 pad 2: +3V3 -> VCC_IO
- C42 pad 1: +3V3 -> VCC_IO
- C43 pad 1: +3V3 -> VCC_IO
- C46 pad 1: +3V3 -> VCC_IO
- C52 pad 2: +3V3 -> VCC_IO
- C53 pad 2: +3V3 -> VCC_IO
- C54 pad 2: +3V3 -> VCC_IO
- C55 pad 2: +3V3 -> VCC_IO
- C56 pad 2: +3V3 -> VCC_IO
- C57 pad 1: +3V3 -> VCC_IO
- C58 pad 1: +3V3 -> VCC_IO
- C59 pad 1: +3V3 -> VCC_IO
- C60 pad 2: +3V3 -> VCC_IO
- C7 pad 1: +3V3 -> VCC_IO
- C8 pad 1: +3V3 -> VCC_IO
- C9 pad 1: +3V3 -> VCC_IO
- J10 pad 8: +3V3 -> VCC_IO
- J11 pad 11: +3V3 -> VCC_IO
- J11 pad 6: unconnected-(J11-Pin_6-Pad6) -> GND
- J11 pad 8: unconnected-(J11-Pin_8-Pad8) -> VCC_IO
- J12 pad 1: +3V3 -> VCC_IO
- J3 pad 2: Out_1 -> Out_2
- J3 pad 3: Out_2 -> Out_1
- J3 pad 5: /STOP_L/STEP -> GND
- J6 pad P2: +3V3 -> VCC_IO
- J6 pad P5: +3V3 -> VCC_IO
- J8 pad 8: +3V3 -> VCC_IO
- J9 pad 11: +3V3 -> VCC_IO
- J9 pad 6: unconnected-(J9-Pin_6-Pad6) -> GND
- J9 pad 8: unconnected-(J9-Pin_8-Pad8) -> VCC_IO
- R2 pad 2: +3V3 -> VCC_IO
- R3 pad 1: +3V3 -> VCC_IO
- R34 pad 2: 5VOUT -> VCC_IO
- R35 pad 2: 5VOUT -> VCC_IO
- R38 pad 1: +3V3 -> VCC_IO
- R42 pad 1: +3V3 -> VCC_IO
- R43 pad 1: +3V3 -> VCC_IO
- R44 pad 1: +3V3 -> VCC_IO
- R5 pad 2: +3V3 -> VCC_IO
- U1 pad 6: +3V3 -> VCC_IO
- U1 pad 7: +3V3 -> VCC_IO
- U3 pad 3: +3V3 -> VCC_IO
- U5 pad 11: +3V3 -> VCC_IO
- U5 pad 12: +3V3 -> VCC_IO
- U6 pad 1: +3V3 -> VCC_IO
- U6 pad 13: +3V3 -> VCC_IO
- U6 pad 19: +3V3 -> VCC_IO
- U6 pad 32: +3V3 -> VCC_IO
- U6 pad 48: +3V3 -> VCC_IO
- U6 pad 64: +3V3 -> VCC_IO
- U8 pad 19: +3V3 -> VCC_IO
- U8 pad 26: +3V3 -> VCC_IO
- U8 pad 37: +3V3 -> VCC_IO
- U8 pad 5: +3V3 -> VCC_IO
- U9 pad 1: +3V3 -> VCC_IO
- U9 pad 19: +3V3 -> VCC_IO
- U9 pad 9: +3V3 -> VCC_IO
Routing:
- net VCC_IO: track 4.42 -> 358.7 mm, vias 1 -> 20
- net +3V3: track 312.1 -> 0.00 mm, vias 19 -> 0
- net INTR: track 0.00 -> 44.2 mm, vias 0 -> 4
- net 5VOUT: track 27.5 -> 67.7 mm
- net Out_1: track 0.20 -> 39.7 mm, vias 0 -> 1
- net Out_2: track 0.00 -> 38.4 mm, vias 0 -> 1
- net DRV_ENN: track 11.1 -> 26.5 mm
- net NSCS_ENC: track 39.0 -> 38.1 mm
- net VS: track 43.1 -> 42.5 mm
- net GND: vias 167 -> 170

Commit message: finished not checked
Parts:
- removed C10, C4, C57, C58, C59, C7: 0.1u, Capacitor_SMD:C_0402_1005Metric
- removed C37: 0.1u, Capacitor_SMD:C_0603_1608Metric_Pad1.08x0.95mm_HandSolder
- removed C42, C43: 22uF, Capacitor_SMD:C_0805_2012Metric_Pad1.18x1.45mm_HandSolder
- removed C44, C45: 2.2u, Capacitor_SMD:C_0402_1005Metric
- removed C46: 4.7u, Capacitor_SMD:C_0402_1005Metric
- removed C47, C48: 15p, Capacitor_SMD:C_0603_1608Metric
- removed C50: 470p, Capacitor_SMD:C_0402_1005Metric
- removed C51: 1u, Capacitor_SMD:C_0402_1005Metric
- removed C52, C53, C54, C56: 10pF, Capacitor_SMD:C_0603_1608Metric_Pad1.08x0.95mm_HandSolder
- removed C55: 0.022uF, Capacitor_SMD:C_0603_1608Metric_Pad1.08x0.95mm_HandSolder
- removed D2: LED_ORANGE, LED_SMD:LED_0402_1005Metric
- removed D3: LED_GREEN, Diode_SMD:D_0402_1005Metric
- removed D8: SP0503BAHT, Package_TO_SOT_SMD:SOT-143
- removed D9: D_Schottky, Diode_SMD:D_MicroSMP_AK
- removed J10, J11: Conn_02x06_Odd_Even, Connector_PinHeader_2.54mm:PinHeader_2x06_P2.54mm_Vertical
- removed J12: Conn_01x02_Pin, Connector_PinHeader_1.27mm:PinHeader_1x02_P1.27mm_Vertical
- removed J13: Conn_01x03_Pin, Connector_PinHeader_1.27mm:PinHeader_1x03_P1.27mm_Vertical
- removed J5: USB_B_Micro, Connector_USB:USB_Micro-B_Molex-105133-0031
- removed J6: JXD2-0Z10NL, JXD2_0Z10NL:JXD2_0Z10NL
- removed R3: 270, Resistor_SMD:R_0402_1005Metric
- removed R32: 12.1k, Resistor_SMD:R_0402_1005Metric
- removed R36, R37: 330, Resistor_SMD:R_0603_1608Metric
- removed R38, R42, R43, R44: 49.9, Resistor_SMD:R_0603_1608Metric
- removed R39, R40, R41: 22, Resistor_SMD:R_0402_1005Metric
- removed U6: STM32H563RGTx, Package_QFP:LQFP-64_10x10mm_P0.5mm
- removed U9: LAN8742A-CZ-TR, LAN8742A_CZ_TR:LAN8742A_CZ_TR
- removed Y2: 25Mhz, Crystal:Crystal_SMD_2016-4Pin_2.0x1.6mm
- R2: value 270 -> 10k; footprint Resistor_SMD:R_0402_1005Metric -> Resistor_SMD:R_0603_1608Metric_Pad0.98x0.95mm_HandSolder; moved to F.Cu
- TH1: moved to B.Cu
- moved R2 52.4 mm to (118.5, 103.7)
- moved TH1 36.9 mm to (103.1, 95.6), turned to 90 degrees
Connections:
- J9 pad 12: unconnected-(J9-Pin_12-Pad12) -> monitoring
- R2 pad 1: Net-(D2-A) -> GND
- R2 pad 2: VCC_IO -> monitoring
- TH1 pad 1: unconnected-(TH1-Pad1) -> monitoring
- TH1 pad 2: unconnected-(TH1-Pad2) -> VCC_IO
Routing:
- net VCC_IO: track 358.7 -> 198.0 mm, vias 20 -> 10
- net LED1: track 62.3 -> 0.00 mm, vias 2 -> 0
- net LED2: track 49.3 -> 0.00 mm, vias 2 -> 0
- net PGOOD1: track 48.6 -> 0.00 mm
- net SPI_MISO_1: track 33.2 -> 0.00 mm
- net SPI_MOSI_1: track 32.1 -> 0.00 mm
- net SCK_1: track 31.1 -> 0.00 mm
- net CSN_1: track 29.3 -> 0.00 mm
- net CLK_EXT_1: track 28.5 -> 0.00 mm
- net D-: track 27.3 -> 0.00 mm
- net Net-(C44-Pad2): track 25.6 -> 0.00 mm, vias 2 -> 0
- net RXP: track 25.3 -> 0.00 mm
- net ETH_TXD1: track 24.6 -> 0.00 mm, vias 2 -> 0
- net RXN: track 24.4 -> 0.00 mm
- net monitoring: track 0.00 -> 23.4 mm, vias 0 -> 1
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Other:
- board size 117.8 x 60 mm -> 60 x 60 mm
- board text removed: "3V3"

Commit message: updated
Parts:
- added Q5: TLP185GR-TPL_SE, TLP185_GR_TPL_SE:TLP185_GR_TPL_SE, B.Cu at (128.9, 105.9)
- added Q6: TLP185GR-TPL_SE, TLP185_GR_TPL_SE:TLP185_GR_TPL_SE, B.Cu at (137.5, 105.9)
- added Q7: TLP185GR-TPL_SE, TLP185_GR_TPL_SE:TLP185_GR_TPL_SE, B.Cu at (120.2, 105.9)
- added R3: 4k7, Resistor_SMD:R_0603_1608Metric_Pad0.98x0.95mm_HandSolder, B.Cu at (102.3, 104.7)
- moved R34 13.4 mm to (123.3, 112.9)
- moved C5 12.3 mm to (140.2, 113.3)
- moved R35 7.54 mm to (129.3, 113.0)
- moved C6 6.30 mm to (135.2, 113.3)
- moved R2 1.83 mm to (118.5, 101.9), turned to -90 degrees
- moved C38 1.17 mm to (118.7, 109.2), turned to 180 degrees
Connections:
- J3 pad 2: Out_2 -> HOME_REF
- J3 pad 4: /IN2/ENC_B -> Out_2
- J3 pad 6: GND -> 12-36V
- J3 pad 7: 5VOUT -> 12-36V
- U8 pad 13: unconnected-(U8-HOME_REF-Pad13) -> HOME_REF
Routing:
- net VCC_IO: track 198.0 -> 188.3 mm
- net Out_1: track 39.7 -> 34.5 mm
- net Out_2: track 38.4 -> 40.1 mm
- net 5VOUT: track 67.7 -> 68.8 mm, vias 2 -> 3
