File: TMCM_1260_alternative_ver_2/TMCM_1260_alternative_ver_2.kicad_pcb (KiCad board)
At the start: 4 copper layers, 60 x 60 mm, 84 parts, among them J1 Motor, J2 CAN, J3 I/O, J4 Power, J8 Conn_02x06_Odd_Even, J9 Conn_02x06_Odd_Even, Q1 NVMFD5C650NLT1G, Q2 NVMFD5C650NLT1G, Q3 NVMFD5C650NLT1G, Q4 NVMFD5C650NLT1G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

Commit message: finished
Parts:
- removed C6: 0.1u, Capacitor_SMD:C_0603_1608Metric
- added C4: 0.1u, Capacitor_SMD:C_0402_1005Metric, F.Cu at (127.9, 104.7)
- added C7: 0.1u, Capacitor_SMD:C_0402_1005Metric, F.Cu at (119.2, 104.6)
- added R26: 24k, Resistor_SMD:R_0402_1005Metric, F.Cu at (131.8, 104.7)
- added R32: 24k, Resistor_SMD:R_0402_1005Metric, F.Cu at (140.4, 104.7)
- added R33: 24k, Resistor_SMD:R_0402_1005Metric, F.Cu at (123.1, 104.7)
- C5: footprint Capacitor_SMD:C_0603_1608Metric -> Capacitor_SMD:C_0402_1005Metric; moved to F.Cu
- R3, R34, R35: footprint Resistor_SMD:R_0603_1608Metric_Pad0.98x0.95mm_HandSolder -> Resistor_SMD:R_0402_1005Metric; moved to F.Cu
- moved R3 23.7 mm to (126.0, 104.7), turned to 0 degrees
- moved R35 14.7 mm to (117.2, 104.7)
- moved R34 13.9 mm to (134.6, 104.7), turned to 0 degrees
- moved C5 9.38 mm to (136.5, 104.7), turned to 0 degrees
- turned Q5 to 180 degrees
- turned Q7 to 180 degrees
Connections:
- C5 pad 1: Out_1 -> STOPR
- J3 pad 2: HOME_REF -> home
- J3 pad 3: Out_1 -> Out_2
- J3 pad 4: Out_2 -> Out_1
- Q1 pad 13: (no net) -> BMB1
- Q1 pad 14: (no net) -> 12-36V
- Q2 pad 13: (no net) -> BMB2
- Q2 pad 14: (no net) -> 12-36V
- Q3 pad 13: (no net) -> BMA1
- Q3 pad 14: (no net) -> 12-36V
- Q4 pad 13: (no net) -> BMA2
- Q4 pad 14: (no net) -> 12-36V
- Q5 pad 1: unconnected-(Q5-Pad1) -> Net-(Q5-Pad1)
- Q5 pad 3: HOME_REF -> home
- Q5 pad 4: unconnected-(Q5-Pad4) -> GND
- Q6 pad 1: unconnected-(Q6-Pad1) -> Net-(Q6-Pad1)
- Q6 pad 4: unconnected-(Q6-Pad4) -> GND
- Q7 pad 1: unconnected-(Q7-Pad1) -> Net-(Q7-Pad1)
- Q7 pad 4: unconnected-(Q7-Pad4) -> GND
- R34 pad 1: Out_2 -> STOPR
- R35 pad 1: Out_1 -> STOPL
- U1 pad PAD: (no net) -> GND
- U8 pad 12: Out_1 -> STOPL
- U8 pad 14: Out_2 -> STOPR
- U8 pad 41: (no net) -> GND
Routing:
- net STOPL: track 0.00 -> 49.3 mm, vias 0 -> 4
- net HOME_REF: track 0.00 -> 43.4 mm, vias 0 -> 3
- net STOPR: track 0.00 -> 36.1 mm, vias 0 -> 3
- net Out_2: track 40.1 -> 10.9 mm
- net Out_1: track 34.5 -> 7.65 mm
- net VCC_IO: track 188.3 -> 208.7 mm, vias 10 -> 8
- net DRV_ENN: track 26.5 -> 20.6 mm
- net 5VOUT: track 68.8 -> 63.8 mm
- net home: track 0.00 -> 3.28 mm
- net SPI_MOSI_DRV: track 18.7 -> 17.7 mm
- net CLK_EXT: track 37.5 -> 37.0 mm
- net Net-(Q7-Pad1): vias 0 -> 1
- net Net-(Q6-Pad1): vias 0 -> 1
- net Net-(Q5-Pad1): vias 0 -> 1
- net GND: vias 122 -> 126
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
Commit message: absolute encoder SPI switched to ABI incremental
Parts:
- added R36: 4k7, Resistor_SMD:R_0402_1005Metric, B.Cu at (130.7, 77.5)
- added R37: 4k7, Resistor_SMD:R_0402_1005Metric, B.Cu at (127.7, 84.9)
- added R38: 4k7, Resistor_SMD:R_0402_1005Metric, B.Cu at (128.7, 84.9)
Connections:
- U5 pad 1: NSCS_ENC -> Net-(U5-CSn)
- U5 pad 14: unconnected-(U5-I/PWM-Pad14) -> INCR_I
- U5 pad 2: SCLK_ENC -> Net-(U5-CLK)
- U5 pad 3: SDI_ENC -> unconnected-(U5-MISO-Pad3)
- U5 pad 4: SDO_ENC -> Net-(U5-MOSI)
- U5 pad 6: unconnected-(U5-B-Pad6) -> INCR_B
- U5 pad 7: unconnected-(U5-A-Pad7) -> INCR_A
- U8 pad 1: NSCS_ENC -> GND
- U8 pad 10: SDI_ENC -> INCR_B
- U8 pad 11: SDO_ENC -> GND
- U8 pad 21: unconnected-(U8-N-Pad21) -> INCR_I
- U8 pad 22: unconnected-(U8-NNEG-Pad22) -> GND
- U8 pad 40: SCLK_ENC -> INCR_A
Routing:
- net SDI_ENC: track 44.9 -> 0.00 mm, vias 1 -> 0
- net INCR_B: track 0.00 -> 44.0 mm, vias 0 -> 1
- net SDO_ENC: track 44.0 -> 0.00 mm, vias 1 -> 0
- net INCR_I: track 0.00 -> 42.4 mm, vias 0 -> 4
- net NSCS_ENC: track 38.1 -> 0.00 mm, vias 1 -> 0
- net SCLK_ENC: track 35.6 -> 0.00 mm, vias 1 -> 0
- net INCR_A: track 0.00 -> 31.8 mm, vias 0 -> 1
- net GND: track 50.3 -> 62.9 mm, vias 126 -> 127
- net Net-(U5-CLK): track 0.00 -> 6.90 mm
- net Net-(U5-MOSI): track 0.00 -> 5.11 mm
- net VCC_IO: track 208.7 -> 211.3 mm, vias 8 -> 10
- net Net-(U5-CSn): track 0.00 -> 1.66 mm
- net SRAL: track 47.0 -> 47.8 mm
- net SRAH: track 45.1 -> 46.0 mm
- net HOME_REF: vias 3 -> 4
