File: TMCM_1260_alternative_ver_2_quilter/TMCM_1260_alternative_ver_2_quilter.kicad_pcb (KiCad board)
At the start: 4 copper layers, 60 x 60 mm, 119 parts, among them J1 Motor, J2 CAN, J3 I/O, J4 Power, J5 USB_B_Micro, J6 JXD2-0Z10NL, J7 Conn_01x05, Q1 NVMFD5C650NLT1G, Q2 NVMFD5C650NLT1G, Q3 NVMFD5C650NLT1G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

Commit message: upload
Parts:
- removed C23: 330u, Capacitor_THT:CP_Radial_D10.0mm_P5.00mm
- removed C4: 0.1u, Capacitor_SMD:C_0603_1608Metric_Pad1.08x0.95mm_HandSolder
- removed J6: JXD2-0Z10NL, JXD2_0Z10NL:JXD2_0Z10NL
- removed J7: Conn_01x05, Connector_PinHeader_2.54mm:PinHeader_1x05_P2.54mm_Vertical
- removed Y1: 8Mhz, digikey-footprints:SMD-2_3.2x2.5mm
- added C41: 47uF, Capacitor_SMD:C_1206_3216Metric, F.Cu at (71.6, 73.4)
- C49, C50, C51, C52, C53, C54, C56, C57, C58, C59, C8, C9, R32, R33, R38, R42, R43, R44, R45, R46, R47, R5, U3, U9: moved to B.Cu
- D8, R26: moved to F.Cu
- H1, H2, H3, H4: renamed from REF**; value MountingHole_3.2mm_M3 -> MountingHole
- moved U8 58.8 mm to (147.4, 89.4)
- moved U4 44.2 mm to (144.3, 76.6)
- moved C14 42.4 mm to (58.8, 100.1)
- moved C25 41.2 mm to (71.2, 135.2)
- moved R34 41.2 mm to (69.9, 141.7)
- moved C26 41.2 mm to (69.8, 131.4)
- moved C27 41.2 mm to (71.6, 131.6)
- moved C38 41.2 mm to (71.5, 138.7)
- moved C16 41.2 mm to (71.2, 136.7)
- moved C28 41.2 mm to (68.0, 131.1)
- moved R35 41.2 mm to (69.9, 140.2)
- moved C22 38.4 mm to (63.5, 72.4)
- moved C12 33.5 mm to (62.6, 91.7)
- moved C13 33.5 mm to (62.6, 89.7)
- moved D1 31.7 mm to (142.3, 68.3)
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Routing:
- net +3V3: track 98.7 -> 0.00 mm, vias 3 -> 0
- net 5VOUT: track 52.9 -> 0.00 mm, vias 3 -> 0
- net SRAL: track 47.0 -> 0.00 mm, vias 3 -> 0
- net SRAH: track 45.1 -> 0.00 mm, vias 3 -> 0
- net GND: track 44.5 -> 0.00 mm, vias 99 -> 12
- net VS: track 43.1 -> 0.00 mm, vias 2 -> 0
- net DRV_ENN: track 25.2 -> 0.00 mm
- net HB1: track 21.5 -> 0.14 mm
- net UART_RX: track 20.3 -> 0.00 mm
- net BMB1: track 116.7 -> 96.9 mm
- net SDI_ENC: track 19.8 -> 0.00 mm
- net BMA1: track 90.8 -> 71.8 mm, vias 2 -> 0
- net HA2: track 19.7 -> 1.34 mm
- net SCLK_ENC: track 18.3 -> 0.00 mm
- net UART_TX: track 18.2 -> 0.00 mm
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