File: ETH_TMC_shield/ETH_TMC_shield.kicad_pcb (KiCad board)
At the start: 4 copper layers, 47.1 x 42.7 mm, 50 parts, among them J10 Conn_02x06_Odd_Even, J11 Conn_02x06_Odd_Even, J12 Conn_01x02_Pin, J13 Conn_01x03_Pin, J5 USB_B_Micro, J6 JXD2-0Z10NL, U6 STM32H563RGTx, U9 LAN8742A-CZ-TR, Y2 25Mhz

Commit message: updated
Routing:
- net +3V3: vias 17 -> 18
Changed lines of the file:
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@@
 		(tags "capacitor")
 		(property "Reference" "C46"
-			(at 1.1684 -0.8128 360)
+			(at 1.1684 -0.8128 0)
 			(layer "F.SilkS")
 			(effects
@@
 		)
 		(property "Value" "4.7u"
-			(at 0 1.16 360)
+			(at 0 1.16 0)
 			(layer "F.Fab")
 			(effects
@@
 		)
 		(fp_text user "${REFERENCE}"
-			(at 0 0 360)
+			(at 0 0 0)
 			(layer "F.Fab")
 			(effects
@@
 		(tags "SOT-143")
 		(property "Reference" "D8"
-			(at 2.0574 -1.2446 90)
+			(at 1.976 1.2752 90)
 			(layer "F.SilkS")
 			(effects
@@
 	)
 	(via
+		(at 83.2892 78.2828)
+		(size 0.4)
+		(drill 0.2)
+		(layers "F.Cu" "B.Cu")
+		(net 1)
+	)
+	(via
 		(at 69.2124 83.6676)
 		(size 0.4)
@@
 	)
 	(segment
-		(start 67.7672 96.8756)
-		(end 70.7644 96.8756)
+		(start 63.3984 98.9584)
+		(end 62.6136 98.9584)
 		(width 0.15)
 		(layer "In2.Cu")
@@
 	)
 	(segment
-		(start 62.7608 98.3208)
-		(end 63.3984 98.9584)
+		(start 67.7672 96.8756)
+		(end 70.7644 96.8756)
 		(width 0.15)
 		(layer "In2.Cu")
@@
 	)
 	(segment
-		(start 59.9948 101.953302)
-		(end 59.9948 98.7272)
+		(start 60.4012 98.3208)
+		(end 61.976 98.3208)
 		(width 0.15)
 		(layer "In2.Cu")
@@
 	)
 	(segment
-		(start 60.4012 98.3208)
-		(end 62.7608 98.3208)
+		(start 59.9948 101.953302)
+		(end 59.9948 98.7272)
 		(width 0.15)
 		(layer "In2.Cu")
@@
 	)
 	(segment
+		(start 62.6136 98.9584)
+		(end 61.976 98.3208)
+		(width 0.15)
+		(layer "In2.Cu")
+		(net 3)
+	)
+	(segment
 		(start 75.1332 95.6564)
 		(end 76.1492 94.6404)
@@
 	)
 	(via
-		(at 59.101391 94.288812)
+		(at 56.6674 95.4786)
 		(size 0.6)
 		(drill 0.3)
@@
 	)
 	(via
-		(at 61.468 97.6884)
+		(at 80.726651 75.9383)
 		(size 0.6)
 		(drill 0.3)
 		(layers "F.Cu" "B.Cu")
-		(free yes)
 		(net 4)
 	)
 	(via
-		(at 80.726651 75.9383)
+		(at 52.0442 80.9572)
 		(size 0.6)
 		(drill 0.3)
@@
 	)
 	(via
-		(at 52.0442 80.9572)
-		(size 0.6)
-		(drill 0.3)
+		(at 60.4012 97.3608)
+		(size 0.4)
+		(drill 0.2)
 		(layers "F.Cu" "B.Cu")
 		(net 4)
@@
 	)
 	(via
-		(at 54.7116 95.6564)
+		(at 54.8386 95.8088)
 		(size 0.6)
 		(drill 0.3)
@@
 	)
 	(segment
-		(start 83.5152 75.8444)
-		(end 83.5152 72.6948)
+		(start 72.5424 64.2112)
+		(end 71.702901 65.050699)
 		(width 0.25)
 		(layer "In2.Cu")
@@
 	)
 	(segment
-		(start 72.5424 64.2112)
-		(end 71.702901 65.050699)
+		(start 81.0006 82.2706)
+		(end 81.0006 78.359)
 		(width 0.25)
 		(layer "In2.Cu")
@@
 	)
 	(segment
+		(start 81.0006 78.359)
+		(end 81.1784 78.1812)
+		(width 0.25)
+		(layer "In2.Cu")
+		(net 73)
+	)
+	(segment
 		(start 71.702901 65.050699)
 		(end 71.702901 65.689001)
@@
 	)
 	(segment
+		(start 83.5152 75.8444)
+		(end 83.8708 75.4888)
+		(width 0.25)
+		(layer "In2.Cu")
+		(net 73)
+	)
+	(segment
 		(start 75.0316 92.9132)
 		(end 79.1464 92.9132)
@@
 	)
 	(segment
+		(start 81.1784 82.4484)
+		(end 81.0006 82.2706)
+		(width 0.25)
+		(layer "In2.Cu")
+		(net 73)
+	)
+	(segment
 		(start 82.042 85.344)
 		(end 82.042 83.312)
@@
 	)
 	(segment
-		(start 71.702901 65.689001)
-		(end 69.9008 67.491102)
+		(start 83.8708 75.4888)
+		(end 83.8708 73.0504)
 		(width 0.25)
 		(layer "In2.Cu")
@@
 	)
 	(segment
-		(start 81.1784 82.4484)
-		(end 81.1784 78.1812)
+		(start 83.8708 73.0504)
+		(end 83.5152 72.6948)
+		(width 0.25)
+		(layer "In2.Cu")
+		(net 73)
+	)
+	(segment
+		(start 71.702901 65.689001)
+		(end 69.9008 67.491102)
 		(width 0.25)
 		(layer "In2.Cu")
@@
 		(hatch edge 0.5)
 		(connect_pads
-			(clearance 0.5)
+			(clearance 0.3)
 		)
 		(min_thickness 0.25)
 		(filled_areas_thickness no)
 		(fill yes
-			(thermal_gap 0.5)
-			(thermal_bridge_width 0.5)
+			(thermal_gap 0.3)
+			(thermal_bridge_width 1)
 		)
 		(polygon

Commit message: finished
Parts:
- moved C46 0.25 mm to (84.0, 78.3)
- moved C7 0.11 mm to (83.6, 90.0)
Connections:
- J10 pad 5: unconnected-(J10-Pin_5-Pad5) -> DRV_ENN_1
Routing:
- net +3V3: track 30.4 -> 28.3 mm
